File: design_blocks_schematics/ad8334.brd (EAGLE design)
At the start: 160 x 100 mm, 68 parts, among them IC1 AD8334ACPZ

Commit message: routing 75% done
Parts:
- removed R12: DNP, resistor:R0603
- removed R14: 1K, resistor:R0603
- added R7: 0R, resistor:R0402
- C19, C20: value 1nF -> 10nF; device rcl:C0402 -> Wurth_Elektronik_Passive_Capacitors_rev18b:WCAP-CSGP_0402
- R1, R3: value 39k -> 39K; device resistor:R0603 -> resistor:R0402
- R10, R11, R13, R2, R8: device resistor:R0603 -> resistor:R0402
- R4, R5: value 4.02k -> 4K02; device resistor:R0805 -> resistor:R0402
- R6: value 274R -> DNP
- R9: value 0R -> 1K; device resistor:R0603 -> resistor:R0402
- moved C53 124.4 mm to (77.8, 34.4), turned to 90 degrees
- moved C54 120.8 mm to (84.3, 39.8), turned to 180 degrees
- moved C56 118.1 mm to (84.3, 44.3), turned to 180 degrees
- moved C55 114.4 mm to (77.8, 49.7), turned to 270 degrees
- moved L29 93.2 mm to (78.0, 30.6), turned to 90 degrees
- moved L32 86.5 mm to (87.3, 44.6), turned to 180 degrees
- moved L30 84.9 mm to (87.1, 39.8), turned to 180 degrees
- moved L31 76.8 mm to (78.1, 53.5), turned to 270 degrees
- moved TP2_GND1 56.6 mm to (83.1, 62.6), turned to 180 degrees
- moved VR2 50.9 mm to (83.3, 30.6), turned to 270 degrees
- moved TP2_8 49.9 mm to (140.2, 17.9)
- moved R1 49.8 mm to (79.7, 30.6), turned to 270 degrees
- moved C19 43.4 mm to (79.0, 34.4), turned to 270 degrees
- moved C20 36.0 mm to (79.0, 49.7), turned to 90 degrees
- moved R3 34.7 mm to (79.7, 53.5), turned to 90 degrees
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Connections:
- removed net N$3: IC1.60, IC1.63, IC1.64, IC1.65
- net +5V: now also R11.2, R2.2, R9.2; no longer R11.1, R14.2, R2.1
- net CLAMP12_1: now also R4.2; no longer R4.1
- net CLAMP12_2: now also R5.2; no longer R5.1
- net EN12: now also R9.1; no longer R13.1
- net EN34: now also R13.1; no longer R14.1
- net GND: now also IC1.60, IC1.63, IC1.64, IC1.65, R10.1, R4.1, R5.1, R6.1; no longer R10.2, R12.2, R4.2, R5.2
- net HILO_12: now also R11.1, R6.2; no longer R11.2, R12.1
- net MODE_12: now also R10.2, R2.1; no longer R10.1, R2.2
- net N$1: now also R7.2; no longer R8.2
- net N$14: no longer R6.1
- net N$15: now also R8.2; no longer R9.2
- net N$2: now also R8.1; no longer R9.1
- net R1_I: now also R7.1; no longer R8.1
- net R1_LO_N: no longer R6.2
Routing:
- net GND: track 8.60 -> 25.3 mm, vias 8 -> 22
- net GAIN12_2: track 0.00 -> 9.39 mm
- net GAIN12_1: track 0.00 -> 8.57 mm
- net INH1: track 8.14 -> 0.00 mm
- net +5V: track 2.20 -> 10.1 mm, vias 2 -> 9
- net VPS1_1: track 0.00 -> 6.71 mm
- net VPS4_1: track 0.00 -> 6.67 mm
- net R1_LO_N1: track 6.35 -> 0.00 mm
- net VPS3_2: track 6.03 -> 0.00 mm
- net HILO_12: track 0.00 -> 6.02 mm
- net EN34: track 0.00 -> 5.28 mm
- net EN12: track 0.00 -> 4.68 mm
- net R1_V1I_N1: track 4.63 -> 0.00 mm
- net CLAMP12_1: track 0.00 -> 4.52 mm
- net CLAMP12_2: track 0.00 -> 4.52 mm
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
Commit message: routing done
Parts:
- added R12: 274R, resistor:R0402
- moved TP2_8 50.4 mm to (92.1, 33.2), turned to 180 degrees
- moved TP2_11 48.9 mm to (92.1, 48.8), turned to 180 degrees
- moved TP2_9 48.9 mm to (92.1, 46.2), turned to 180 degrees
- moved TP2_7 48.7 mm to (92.1, 35.8), turned to 180 degrees
- moved TP2_12 48.6 mm to (92.1, 51.4), turned to 180 degrees
- moved TP2_6 48.1 mm to (92.1, 38.4), turned to 180 degrees
- moved TP2_10 47.7 mm to (92.1, 43.6), turned to 180 degrees
- moved TP2_5 47.7 mm to (92.1, 41.0), turned to 180 degrees
- moved TP2_GND1 33.2 mm to (92.1, 30.6)
- moved C14 7.09 mm to (95.5, 49.5)
- moved C13 6.93 mm to (95.5, 50.7)
- moved C6 6.35 mm to (95.5, 35.1)
- moved C18 6.08 mm to (95.5, 44.3)
- moved C4 6.08 mm to (95.5, 39.1)
- moved C7 6.03 mm to (95.5, 33.9)
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Connections:
- net N$14: now also R12.1
- net R1_LO_N: now also R12.2
Routing:
- net R1_V2I_P: track 0.00 -> 23.4 mm, vias 0 -> 2
- net R1_V2I_N: track 0.00 -> 21.9 mm, vias 0 -> 2
- net R2_V2I_P: track 1.12 -> 22.7 mm, vias 1 -> 2
- net R2_V2I_N: track 1.12 -> 21.5 mm, vias 1 -> 2
- net R2_V2O_P: track 0.00 -> 16.3 mm
- net R1_V2O_P: track 0.00 -> 16.1 mm
- net R2_V2O_N: track 0.00 -> 15.4 mm
- net R1_V2O_N: track 0.00 -> 15.2 mm
- net R2_V1O_N: track 0.00 -> 14.8 mm
- net R1_V1O_N: track 0.00 -> 14.7 mm
- net R2_V1O_P: track 0.00 -> 13.9 mm
- net R1_V1O_P: track 0.00 -> 13.9 mm
- net GND: track 25.3 -> 35.3 mm, vias 22 -> 31
- net VPS12_1: track 0.00 -> 5.48 mm
- net VPS34_1: track 0.00 -> 5.48 mm
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