File: design_blocks_schematics/ad8334.brd (EAGLE design)
At the start: 160 x 100 mm, 68 parts, among them IC1 AD8334ACPZ

Commit message: updated input/output net names
Connections:
- net LVOUT_0 renamed IN_A
- net LVOUT_1 renamed IN_B
- net R1_OUT_N renamed OUT_B_N
- net R1_OUT_P renamed OUT_B_P
- net R2_OUT_N renamed OUT_A_N
- net R2_OUT_P renamed OUT_A_P
- net VCM1 renamed OUT_A_VCM
- net VCM3 renamed OUT_B_VCM
Changed lines of the file:
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@@
 <wire x1="84.3024" y1="44.5976" x2="83.8" y2="45.1" width="0.2" layer="1"/>
 </signal>
-<signal name="VCM1">
+<signal name="OUT_A_VCM">
 <contactref element="IC1" pad="50"/>
 </signal>
@@
 <wire x1="68.8" y1="34.6" x2="68.8" y2="36.4" width="0.2" layer="1"/>
 </signal>
-<signal name="LVOUT_1" class="2">
-<contactref element="D2" pad="3"/>
-<contactref element="L6" pad="1"/>
-<wire x1="62.4" y1="33.6" x2="65.2" y2="33.6" width="0.2" layer="1"/>
-</signal>
 <signal name="VPS1_1">
 <contactref element="IC1" pad="55"/>
@@
 <wire x1="77.0976" y1="51.4976" x2="78.1" y2="52.5" width="0.2" layer="1"/>
 </signal>
-<signal name="LVOUT_0">
+<signal name="IN_A">
 <contactref element="D1" pad="3"/>
 <contactref element="L1" pad="1"/>
@@
 <wire x1="74.8" y1="49" x2="75" y2="49.2" width="0.2" layer="1"/>
 </signal>
-<signal name="R1_OUT_N">
+<signal name="OUT_B_N">
 <contactref element="C6" pad="2"/>
 </signal>
-<signal name="R1_OUT_P">
+<signal name="OUT_B_P">
 <contactref element="C7" pad="2"/>
 </signal>
@@
 <wire x1="70" y1="40.1" x2="70" y2="39.6" width="0.2" layer="1"/>
 </signal>
-<signal name="R2_OUT_P">
+<signal name="OUT_A_P">
 <contactref element="C13" pad="2"/>
 </signal>
-<signal name="R2_OUT_N">
+<signal name="OUT_A_N">
 <contactref element="C14" pad="2"/>
 </signal>
@@
 <wire x1="74.3" y1="35.45" x2="73.9" y2="35.05" width="0.2" layer="1"/>
 </signal>
-<signal name="VCM3">
+<signal name="OUT_B_VCM">
 <contactref element="IC1" pad="30"/>
 </signal>
@@
 <via x="75.8" y="43.3" extent="1-16" drill="0.35"/>
 </signal>
+<signal name="IN_B" class="2">
+<contactref element="D2" pad="3"/>
+<contactref element="L6" pad="1"/>
+<wire x1="62.4" y1="33.6" x2="65.2" y2="33.6" width="0.2" layer="1"/>
+</signal>
 </signals>
