File: design_blocks_schematics/ad8334.sch (EAGLE design)
At the start: 68 parts, among them IC1 AD8334ACPZ

Commit message: routing 75% done
Parts:
- removed R12: DNP, resistor:R-EU_R0603
- removed R14: 1K, resistor:R-EU_R0603
- added R7: 0R, resistor:R-EU_R0402
- C19, C20: value 1nF -> 10nF; device rcl:C-EUC0402 -> Wurth_Elektronik_Passive_Capacitors_rev18b:WCAP-CSGP_0402_885012205037
- R1, R3: value 39k -> 39K; device resistor:R-EU_R0603 -> resistor:R-EU_R0402
- R10, R11, R13, R2, R8: device resistor:R-EU_R0603 -> resistor:R-EU_R0402
- R4, R5: value 4.02k -> 4K02; device resistor:R-EU_R0805 -> resistor:R-EU_R0402
- R6: value 274R -> DNP
- R9: value 0R -> 1K; device resistor:R-EU_R0603 -> resistor:R-EU_R0402
Connections:
- removed net N$3: IC1.COM1, IC1.COM2, IC1.GND_(EP), IC1.NC_5
- net +5V: now also R11.2, R2.2, R9.2; no longer R11.1, R14.2, R2.1
- net CLAMP12_1: now also R4.2; no longer R4.1
- net CLAMP12_2: now also R5.2; no longer R5.1
- net EN12: now also R9.1; no longer R13.1
- net EN34: now also R13.1; no longer R14.1
- net GND: now also IC1.COM1, IC1.COM2, IC1.GND_(EP), IC1.NC_5, R10.1, R4.1, R5.1, R6.1; no longer R10.2, R12.2, R4.2, R5.2
- net HILO_12: now also R11.1, R6.2; no longer R11.2, R12.1
- net MODE_12: now also R10.2, R2.1; no longer R10.1, R2.2
- net N$1: now also R7.2; no longer R8.2
- net N$14: no longer R6.1
- net N$15: now also R8.2; no longer R9.2
- net N$2: now also R8.1; no longer R9.1
- net R1_I: now also R7.1; no longer R8.1
- net R1_LO_N: no longer R6.2
Other:
- moved on the sheet: R10, R11, R13, R2, R4, R5, R6, R8, R9

Commit message: routing done
Parts:
- added R12: 274R, resistor:R-EU_R0402
Connections:
- net N$14: now also R12.1
- net R1_LO_N: now also R12.2
Changed lines of the file:
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@@
 <part name="R6" library="resistor" library_urn="urn:adsk.eagle:library:348" deviceset="R-EU_" device="R0402" package3d_urn="urn:adsk.eagle:package:26058/2" value="DNP"/>
 <part name="R10" library="resistor" library_urn="urn:adsk.eagle:library:348" deviceset="R-EU_" device="R0402" package3d_urn="urn:adsk.eagle:package:26058/2" value="DNP"/>
+<part name="R12" library="resistor" library_urn="urn:adsk.eagle:library:348" deviceset="R-EU_" device="R0402" package3d_urn="urn:adsk.eagle:package:26058/2" value="274R"/>
 </parts>
 <sheets>
@@
 <attribute name="NAME" x="158.75" y="29.4386" size="1.778" layer="95"/>
 <attribute name="VALUE" x="158.75" y="27.178" size="1.778" layer="96"/>
+</instance>
+<instance part="R12" gate="G$1" x="99.06" y="86.36" smashed="yes" rot="R90">
+<attribute name="NAME" x="95.25" y="87.4014" size="1.778" layer="95" rot="R180"/>
+<attribute name="VALUE" x="95.25" y="84.582" size="1.778" layer="96" rot="R180"/>
 </instance>
 </instances>
@@
 <junction x="99.06" y="93.98"/>
 <label x="114.3" y="93.98" size="1.778" layer="95"/>
+<pinref part="R12" gate="G$1" pin="2"/>
 </segment>
 </net>
@@
 <wire x1="99.06" y1="81.28" x2="99.06" y2="78.74" width="0.1524" layer="91"/>
 <pinref part="C12" gate="G$1" pin="2"/>
-</segment>
-</net>
+<pinref part="R12" gate="G$1" pin="1"/>
+</segment>
+</net>
