File: design_blocks_schematics/ltc2344-16.brd (EAGLE design)
At the start: 6 parts

Commit message: update on adc
Parts:
- C140: value 47uf -> 47uf 6.3V; device rcl:C1210 -> rcl:C0603
Connections:
- net 5V renamed +5V
- net OVDD renamed N$1
Changed lines of the file:
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@@
 <setting verticaltext="up"/>
 </settings>
-<grid distance="50" unitdist="mil" unit="mil" style="lines" multiple="1" display="no" altdistance="5" altunitdist="mil" altunit="mil"/>
+<grid distance="50" unitdist="mil" unit="mil" style="lines" multiple="1" display="yes" altdistance="5" altunitdist="mil" altunit="mil"/>
 <layers>
 <layer number="1" name="Top" color="4" fill="1" visible="yes" active="yes"/>
@@
 <attribute name="VALUE" x="-10.795" y="-27.305" size="1.27" layer="27"/>
 </element>
-<element name="C140" library="rcl" library_urn="urn:adsk.eagle:library:334" package="C1210" package3d_urn="urn:adsk.eagle:package:23619/2" value="47uf" x="1.27" y="-16.51" smashed="yes">
+<element name="C140" library="rcl" library_urn="urn:adsk.eagle:library:334" package="C0603" package3d_urn="urn:adsk.eagle:package:23616/2" value="47uf 6.3V" x="1.27" y="-16.51" smashed="yes">
 <attribute name="NAME" x="-0.635" y="-14.605" size="1.27" layer="25"/>
-<attribute name="POPULARITY" value="0" x="-17.78" y="-21.59" size="1.778" layer="27" display="off"/>
+<attribute name="POPULARITY" value="73" x="-17.78" y="-21.59" size="1.778" layer="27" display="off"/>
 <attribute name="SPICEPREFIX" value="C" x="-17.78" y="-21.59" size="1.778" layer="27" display="off"/>
 <attribute name="VALUE" x="-0.635" y="-19.685" size="1.27" layer="27"/>
@@
 <signal name="GND" class="2">
 <contactref element="ADC1" pad="9"/>
-<contactref element="ADC1" pad="20"/>
-<contactref element="ADC1" pad="29"/>
-<contactref element="C141" pad="2"/>
-<contactref element="C143" pad="2"/>
 <contactref element="C139" pad="2"/>
 <contactref element="ADC1" pad="11"/>
@@
 <contactref element="ADC1" pad="13"/>
 <contactref element="ADC1" pad="14"/>
-<contactref element="ADC1" pad="EXP"/>
-<contactref element="ADC1" pad="32"/>
+<contactref element="ADC1" pad="29"/>
+<contactref element="ADC1" pad="20"/>
+<contactref element="C143" pad="2"/>
+<contactref element="C141" pad="2"/>
 <contactref element="ADC1" pad="31"/>
 <contactref element="C142" pad="2"/>
+<contactref element="ADC1" pad="32"/>
+<contactref element="ADC1" pad="EXP"/>
 <wire x1="-9.51" y1="-25.4" x2="-9.51" y2="-30.48" width="0" layer="19" extent="1-1"/>
 <wire x1="-9.37" y1="-20.08" x2="-9.51" y2="-25.4" width="0" layer="19" extent="1-1"/>
@@
 <wire x1="-6.87" y1="-20.08" x2="-7.37" y2="-20.08" width="0" layer="19" extent="1-1"/>
 <wire x1="-7.62" y1="-17.78" x2="-7.37" y2="-20.08" width="0" layer="19" extent="1-1"/>
-<wire x1="-5.32" y1="-18.03" x2="-7.62" y2="-17.78" width="0" layer="19" extent="1-1"/>
 <wire x1="-7.87" y1="-15.48" x2="-7.62" y2="-17.78" width="0" layer="19" extent="1-1"/>
 <wire x1="-8.87" y1="-15.48" x2="-7.87" y2="-15.48" width="0" layer="19" extent="1-1"/>
 <wire x1="-9.37" y1="-15.48" x2="-8.87" y2="-15.48" width="0" layer="19" extent="1-1"/>
+<wire x1="-5.32" y1="-18.03" x2="-7.62" y2="-17.78" width="0" layer="19" extent="1-1"/>
 <wire x1="-3.16" y1="-30.48" x2="-9.51" y2="-30.48" width="0" layer="19" extent="1-1"/>
 <wire x1="-3.16" y1="-25.4" x2="-3.16" y2="-30.48" width="0" layer="19" extent="1-1"/>
-<wire x1="2.67" y1="-16.51" x2="-5.32" y2="-18.03" width="0" layer="19" extent="1-1"/>
+<wire x1="2.12" y1="-16.51" x2="-5.32" y2="-18.03" width="0" layer="19" extent="1-1"/>
 </signal>
 <signal name="N$81">
@@
 <contactref element="ADC1" pad="12"/>
 <contactref element="C140" pad="1"/>
-<wire x1="-0.13" y1="-16.51" x2="-7.87" y2="-20.08" width="0" layer="19" extent="1-1"/>
+<wire x1="0.42" y1="-16.51" x2="-7.87" y2="-20.08" width="0" layer="19" extent="1-1"/>
 </signal>
 <signal name="CNV">
@@
 <contactref element="ADC1" pad="17"/>
 </signal>
-<signal name="SDO1">
-<contactref element="ADC1" pad="18"/>
-</signal>
 <signal name="SDO2">
 <contactref element="ADC1" pad="23"/>
@@
 <contactref element="ADC1" pad="1"/>
 </signal>
-<signal name="OVDD">
-<contactref element="C143" pad="1"/>
-<contactref element="ADC1" pad="21"/>
-<wire x1="-5.32" y1="-17.53" x2="-4.46" y2="-30.48" width="0" layer="19" extent="1-1"/>
-</signal>
-<signal name="5V">
+<signal name="+5V">
 <contactref element="ADC1" pad="30"/>
 <contactref element="C142" pad="1"/>
 <wire x1="-8.37" y1="-15.48" x2="-10.81" y2="-30.48" width="0" layer="19" extent="1-1"/>
 </signal>
+<signal name="N$1">
+<contactref element="ADC1" pad="21"/>
+<contactref element="C143" pad="1"/>
+<wire x1="-5.32" y1="-17.53" x2="-4.46" y2="-30.48" width="0" layer="19" extent="1-1"/>
+</signal>
+<signal name="SDO1">
+<contactref element="ADC1" pad="18"/>
+</signal>
 </signals>
