File: design_blocks_schematics/lt8471.brd (EAGLE design)
At the start: 160 x 100 mm, 24 parts, among them IC2 LT8471EFE#PBF

Commit message: cleanup schematic/WIP layout
Parts:
- R5: value 261k 25V -> 220k 25V
- R6: value 82k 25V -> 56k 25V
- moved R6 7.58 mm to (79.3, 21.6), turned to 90 degrees
- moved R5 3.01 mm to (76.3, 21.6), turned to 270 degrees
- moved R18 0.29 mm to (81.8, 21.6)
Connections:
- net N5V renamed -5V
- net P5V renamed +5V
- net RT renamed N$1
- net VIN1 renamed VIN
- removed net OV/UV: IC2.6, R5.2
- new net N$4: IC2.6, R5.1, R6.2
- net VCC: now also R5.2; no longer R5.1, R6.2
Routing:
- net N$4: track 0.00 -> 15.7 mm
- net +5V: track 15.6 -> 0.00 mm, vias 2 -> 0
- net VCC: track 11.2 -> 0.00 mm, vias 5 -> 4
- net OV/UV: track 9.48 -> 0.00 mm
- net GND: track 6.25 -> 0.00 mm, vias 20 -> 16
- net VIN: track 23.8 -> 22.7 mm
- net N$1: track 8.32 -> 7.36 mm
- added copper zone on layer 1, net N5V
- added copper zone on layer 1, net P5V
- removed copper zone on layer 1, net +5V
- removed copper zone on layer 1, net -5V
