File: silense.brd (EAGLE design)
At the start: 160 x 100 mm, 192 parts, among them IC1 AD8334ACPZ, J1 FMC-LPC

Commit message: update: - some more todos - output connector added - input connections (16 channels)
Parts:
- removed U$1: HIROSE_FH28-68S-05SH05, wouter:HIROSE_FH28E-68S-05SH05
- added C1, C2, C3, C4, C6, C7: 0.1uF, Wurth_Elektronik_Passive_Capacitors_rev18b:WCAP-CSGP_0402
- added C30: CBEC219-3479B001C1AF, wouter:BTB_CONN_68_F
- C10, C5, C8, C9: value o.1uF -> 0.1uF
- moved LVOUT_0 123.3 mm to (-19.1, 78.7)
- moved VDDP$1 102.9 mm to (-19.1, 95.2)
- moved D5_0 101.6 mm to (-15.2, 168.9)
- moved D6_1 101.6 mm to (-30.5, 168.9)
- moved D5_1 101.6 mm to (-20.3, 168.9)
- moved D6_0 101.6 mm to (-25.4, 168.9)
- moved C139 100.3 mm to (-25.4, 160.0)
- moved C141 100.3 mm to (-31.8, 160.0)
- moved D12 100.3 mm to (-17.8, 160.0)
- moved R47 99.1 mm to (-17.8, 163.8)
- moved R48 99.1 mm to (-27.9, 163.8)
- moved D14 99.1 mm to (-19.1, 154.9)
- moved D17 99.1 mm to (-27.9, 154.9)
- moved TP2_6 92.7 mm to (-15.2, 148.6)
- moved TP2_8 92.7 mm to (-27.9, 148.6)
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Connections:
- removed net INH3: C23.1, C24.2, C25.1
- removed net LO3_N: R6.1
- removed net LO4_N: R7.1
- removed net R2_1: IC1.1
- new net 3P3V: J1.C39, J1.D40
- new net IN0_0: J1.G6, STHV_0.IN1_0
- new net IN0_1: J1.G7, STHV_0.IN1_1
- new net IN10_0: J1.G21
- new net IN10_1: J1.G22
- new net IN11_0: J1.H22
- new net IN11_1: J1.H23
- new net IN12_0: J1.G24
- new net IN12_1: J1.G25
- new net IN13_0: J1.H25
- new net IN13_1: J1.H26
- new net IN14_0: J1.G27
- new net IN14_1: J1.G28
- new net IN15_0: J1.H28
- new net IN15_1: J1.H29
- new net IN9_0: J1.H19
- new net IN9_1: J1.H20
- new net INH2: C23.1, C24.2, C25.1, IC1.1
- new net LA28_N: J1.H32
- new net LA28_P: J1.H31
- new net LA30_N: J1.H35
- new net LA30_P: J1.H34
- new net LA32_N: J1.H38
- new net LA32_P: J1.H37
- new net N$15: C12.1
- new net OUT_10: C30.12
- new net OUT_11: C30.13
- new net OUT_12: C30.14
- new net OUT_13: C30.15
- new net OUT_14: C30.16
- new net OUT_15: C30.17
- new net OUT_16: C30.18
- new net OUT_17: C30.19
- new net OUT_18: C30.20
- new net OUT_19: C30.21
- new net OUT_20: C30.22
- new net OUT_21: C30.23
- new net OUT_22: C30.24
- new net OUT_23: C30.25
- new net OUT_24: C30.26
- new net OUT_25: C30.27
- new net OUT_26: C30.28
- new net OUT_27: C30.29
- new net OUT_28: C30.30
- new net OUT_29: C30.31
- new net OUT_30: C30.32
- new net OUT_31: C30.33
- new net OUT_32: C30.36
- new net OUT_33: C30.37
- new net OUT_34: C30.38
- new net OUT_35: C30.39
- new net OUT_36: C30.40
- new net OUT_37: C30.41
- new net OUT_38: C30.42
- new net OUT_39: C30.43
- new net OUT_40: C30.44
- new net OUT_41: C30.45
- new net OUT_42: C30.46
- new net OUT_43: C30.47
- new net OUT_44: C30.48
- new net OUT_45: C30.49
- new net OUT_46: C30.50
- new net OUT_47: C30.51
- new net OUT_48: C30.52
- new net OUT_49: C30.53
- new net OUT_50: C30.54
- new net OUT_51: C30.55
- new net OUT_52: C30.56
- new net OUT_53: C30.57
- new net OUT_54: C30.58
- new net OUT_55: C30.59
- new net OUT_56: C30.60
- new net OUT_57: C30.61
- new net OUT_58: C30.62
- new net OUT_59: C30.63
- new net OUT_60: C30.64
- new net OUT_61: C30.65
- new net OUT_62: C30.66
- new net OUT_63: C30.67
- new net OUT_8: C30.10
- new net OUT_9: C30.11
- net GND: now also C30.1, C30.34, C30.35, C30.68, C5.2, J1.C1, J1.C12, J1.C13, J1.C16, J1.C17, J1.C20, J1.C21, J1.C24, J1.C25, J1.C28, J1.C29, J1.C32, J1.C33, J1.C36, J1.C38, J1.C4, J1.C40, J1.C5, J1.C8, J1.C9, J1.D10, J1.D13, J1.D16, J1.D19, J1.D2, J1.D22, J1.D25, J1.D28, J1.D3, J1.D37, J1.D39, J1.D6, J1.D7, J1.G1, J1.G11, J1.G14, J1.G17, J1.G20, J1.G23, J1.G26, J1.G29, J1.G32, J1.G35, J1.G38, J1.G4, J1.G40, J1.G5, J1.G8, J1.H12, J1.H15, J1.H18, J1.H21, J1.H24, J1.H27, J1.H3, J1.H30, J1.H33, J1.H36, J1.H39, J1.H6, J1.H9; no longer C5.1
- net IN1_0: now also J1.H7, STHV_0.IN2_0; no longer STHV_0.IN1_0
- net IN1_1: now also J1.H8, STHV_0.IN2_1; no longer STHV_0.IN1_1
- net IN2_0: now also J1.G9, STHV_0.IN3_0; no longer STHV_0.IN2_0
- net IN2_1: now also J1.G10, STHV_0.IN3_1; no longer STHV_0.IN2_1
- net IN3_0: now also J1.H10, STHV_0.IN4_0; no longer STHV_0.IN3_0
- net IN3_1: now also J1.H11, STHV_0.IN4_1; no longer STHV_0.IN3_1
- net IN4_0: now also J1.G12, STHV_0.IN5_0; no longer STHV_0.IN4_0
- net IN4_1: now also J1.G13, STHV_0.IN5_1; no longer STHV_0.IN4_1
- net IN5_0: now also J1.H13, STHV_0.IN6_0; no longer STHV_0.IN5_0
- net IN5_1: now also J1.H14, STHV_0.IN6_1; no longer STHV_0.IN5_1
- net IN6_0: now also J1.G15, STHV_0.IN7_0; no longer STHV_0.IN6_0
- net IN6_1: now also J1.G16, STHV_0.IN7_1; no longer STHV_0.IN6_1
- net IN7_0: now also J1.H16, STHV_0.IN8_0; no longer STHV_0.IN7_0
- net IN7_1: now also J1.H17, STHV_0.IN8_1; no longer STHV_0.IN7_1
- net IN8_0: now also J1.G18; no longer STHV_0.IN8_0
- net IN8_1: now also J1.G19; no longer STHV_0.IN8_1
- net INH4: now also IC1.16
- net N$1: now also C5.1; no longer C5.2
- net OUT_0: now also C30.2
- net OUT_1: now also C30.3
- net OUT_2: now also C30.4
- net OUT_3: now also C30.5
- net OUT_4: now also C30.6
- net OUT_5: now also C30.7
- net OUT_6: now also C30.8
- net OUT_7: now also C30.9
- net R1_LO_N: now also C1.1, IC1.13, R7.1; no longer C12.1
- net R1_LO_P: now also C2.1, IC1.12
- net R1_V2I_N: now also C1.2
- net R1_V2I_P: now also C2.2
- net R1_V2O_N: now also C4.1
- net R1_V2O_P: now also C3.1
- net R2_LO_N: now also R6.1
- net R2_V2O_N: now also C6.1
- net R2_V2O_P: now also C7.1

Commit message: added powerblock for +-5V
Parts:
- added C39: C3216X7R1H225K160AE, samacsys:CAPC3216X180N
- added C40, C43, C44, C47: 1206 x7r 47uF 25V, samacsys:CAPC6050X550N
- added C41, C42: 0.1uF x7r 1206, samacsys:CAPC3416X90N
- added C45, C46: 1206 x7r 2.2uF 25V, rcl:C1206
- added D25: MBRS360T3G, samacsys:DIOM7958X256N
- added D26: VS-MBRS340-M3_9AT, samacsys:DIOM7959X262N
- added IC3: LT8471EFE#PBF, samacsys:SOP65P640X120-21N
- added L2: 744025150, samacsys:WE-TPC_282892
- added L7: 74437324068, samacsys:WE-LHMI_402048
- added L8: 74437324100, samacsys:WE-LHMI_402048
- added R17: 261k 25V, resistor:M1206
- added R18: 82k 25V, resistor:M1206
- added R19, R21: 316k, rcl:R1206
- added R20, R22: 59k, rcl:R1206
- added R23, R24: 100k, rcl:R1206
- added R25: 187k, rcl:R1206
- moved C191 215.7 mm to (49.5, 20.3)
- moved C190 204.8 mm to (50.8, 26.7)
- moved C189 194.8 mm to (50.8, 29.2)
- moved C179 186.1 mm to (52.1, 94.0)
- moved C178 184.8 mm to (61.0, 94.0)
- moved C188 184.2 mm to (50.8, 33.0)
- moved C185 177.3 mm to (67.3, 25.4)
- moved C177 175.6 mm to (61.0, 90.2)
- moved C187 173.7 mm to (50.8, 36.8)
- moved C184 168.0 mm to (68.6, 29.2)
- moved C176 167.0 mm to (61.0, 85.1)
- moved C174 163.1 mm to (74.9, 77.5)
- moved C186 162.4 mm to (50.8, 41.9)
- moved C175 162.3 mm to (64.8, 80.0)
- moved C183 157.7 mm to (68.6, 33.0)
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Connections:
- new net C3: IC3.13, L2.1
- new net E1: D26.1, IC3.2, L7.1
- new net E2: D25.1, IC3.19, L8.2
- new net FB1: IC3.5, R19.1, R20.2
- new net FB2: IC3.16, R21.1, R22.2
- new net N3V3: C44.2, D25.2, R21.2
- new net OV/UV: IC3.6, R17.2
- new net P3V3: C43.2, L7.2, R19.2
- new net PG1: IC3.4, R24.1
- new net PG2: IC3.17, R23.2
- new net RT: IC3.7, R25.1
- new net SS1: C41.2, IC3.8
- new net SS2: C42.1, IC3.15
- new net VINPOS: C40.2, C45.1, C46.2, IC3.1, IC3.20, L2.2, R17.1, R18.2, R23.1, R24.2
- new net VINT: C39.1, C47.1, IC3.14, IC3.18, IC3.3
- net GND: now also C39.2, C40.1, C41.1, C42.2, C43.1, C44.1, C45.2, C46.1, C47.2, D26.2, IC3.10, IC3.11, IC3.12, IC3.21, IC3.9, L8.1, R18.1, R20.1, R22.1, R25.2

Commit message: updated values and connections for +-5V
Connections:
- net N3V3 renamed N5V
- net P3V3 renamed P5V
- removed net VINPOS: C40.2, C45.1, C46.2, IC3.1, IC3.20, L2.2, R17.1, R18.2, R23.1, R24.2
- net HVP_CW: now also C40.2, C45.1, C46.2, IC3.1, IC3.20, L2.2, R17.1, R18.2, R23.1, R24.2
Changed lines of the file:
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@@
 <contactref element="D20" pad="C"/>
 <contactref element="POWER_BOARD_CONN" pad="P$2"/>
+<contactref element="C40" pad="2"/>
+<contactref element="R18" pad="2"/>
+<contactref element="R17" pad="1"/>
+<contactref element="L2" pad="2"/>
+<contactref element="R24" pad="2"/>
+<contactref element="R23" pad="1"/>
+<contactref element="C45" pad="1"/>
+<contactref element="C46" pad="2"/>
+<contactref element="IC3" pad="1"/>
+<contactref element="IC3" pad="20"/>
 <wire x1="61.91" y1="90.17" x2="61.91" y2="93.98" width="0" layer="19" extent="1-1"/>
 <wire x1="53.02" y1="93.98" x2="61.91" y2="93.98" width="0" layer="19" extent="1-1"/>
 <wire x1="57.04" y1="57.005" x2="61.91" y2="90.17" width="0" layer="19" extent="1-1"/>
 <wire x1="64.45" y1="55.88" x2="57.04" y2="57.005" width="0" layer="19" extent="1-1"/>
+<wire x1="98.71" y1="-52.139" x2="64.45" y2="55.88" width="0" layer="19" extent="1-1"/>
+<wire x1="98.785" y1="-57.245" x2="98.71" y2="-52.139" width="0" layer="19" extent="1-1"/>
+<wire x1="104.635" y1="-57.245" x2="98.785" y2="-57.245" width="0" layer="19" extent="1-1"/>
+<wire x1="104.61" y1="-55.139" x2="104.635" y2="-57.245" width="0" layer="19" extent="1-1"/>
+<wire x1="109.31" y1="-64.07" x2="104.635" y2="-57.245" width="0" layer="19" extent="1-1"/>
+<wire x1="112.71" y1="-67.27" x2="109.31" y2="-64.07" width="0" layer="19" extent="1-1"/>
+<wire x1="107.21" y1="-69.32" x2="109.31" y2="-64.07" width="0" layer="19" extent="1-1"/>
+<wire x1="101.61" y1="-70.78" x2="107.21" y2="-69.32" width="0" layer="19" extent="1-1"/>
+<wire x1="116.032" y1="-61.67" x2="112.71" y2="-67.27" width="0" layer="19" extent="1-1"/>
+<wire x1="116.032" y1="-59.17" x2="116.032" y2="-61.67" width="0" layer="19" extent="1-1"/>
 <wire x1="-53.66" y1="154.94" x2="53.02" y2="93.98" width="0" layer="19" extent="1-1"/>
 <wire x1="-69.62" y1="10.55" x2="57.04" y2="57.005" width="0" layer="19" extent="1-1"/>
@@
 <contactref element="J1" pad="G28"/>
 </signal>
-<signal name="VINPOS" class="2">
-<contactref element="R17" pad="1"/>
-<contactref element="L2" pad="2"/>
-<contactref element="R24" pad="2"/>
-<contactref element="R23" pad="1"/>
-<contactref element="R18" pad="2"/>
-<contactref element="C40" pad="2"/>
-<contactref element="C45" pad="1"/>
-<contactref element="C46" pad="2"/>
-<contactref element="IC3" pad="1"/>
-<contactref element="IC3" pad="20"/>
-<wire x1="116.032" y1="-61.67" x2="116.032" y2="-59.17" width="0" layer="19" extent="1-1"/>
-<wire x1="112.71" y1="-67.27" x2="116.032" y2="-61.67" width="0" layer="19" extent="1-1"/>
-<wire x1="109.31" y1="-64.07" x2="112.71" y2="-67.27" width="0" layer="19" extent="1-1"/>
-<wire x1="107.21" y1="-69.32" x2="109.31" y2="-64.07" width="0" layer="19" extent="1-1"/>
-<wire x1="101.61" y1="-70.78" x2="107.21" y2="-69.32" width="0" layer="19" extent="1-1"/>
-<wire x1="104.635" y1="-57.245" x2="109.31" y2="-64.07" width="0" layer="19" extent="1-1"/>
-<wire x1="104.61" y1="-55.139" x2="104.635" y2="-57.245" width="0" layer="19" extent="1-1"/>
-<wire x1="98.785" y1="-57.245" x2="104.635" y2="-57.245" width="0" layer="19" extent="1-1"/>
-<wire x1="98.71" y1="-52.139" x2="98.785" y2="-57.245" width="0" layer="19" extent="1-1"/>
-</signal>
-<signal name="P3V3" class="2">
+<signal name="P5V" class="2">
 <contactref element="R19" pad="2"/>
 <contactref element="L7" pad="2"/>
@@
 <wire x1="85.01" y1="-49.13" x2="89.96" y2="-57.57" width="0" layer="19" extent="1-1"/>
 </signal>
-<signal name="N3V3" class="2">
+<signal name="N5V" class="2">
 <contactref element="D25" pad="2"/>
 <contactref element="R21" pad="2"/>

Commit message: updated hierarchy to 16 ch
Parts:
- removed ADC1: LTC2344-16, wouter:QFN32
- removed C1, C10, C11, C12, C13, C14, C15, C16, C17, C18, C2, C21, C22, C23, C26, C3, C4, C5, C51, C52, C53, C54, C55, C56, C6, C7, C8, C9: 0.1uF, Wurth_Elektronik_Passive_Capacitors_rev18b:WCAP-CSGP_0402
- removed C139, C142, C143: 0.1uf, rcl:C0402
- removed C140: 47uf, rcl:C1210
- removed C141: 2.2uf, rcl:C0402
- removed C170, C171, C172, C173, C174, C175, C176, C177, C178, C179, C180, C181, C182, C183, C184, C185, C186, C187, C188, C189, C190, C191: 220n 100V, rcl:C0805
- removed C19, C20: 1nF, rcl:C0402
- removed C24, C27: 22pF, Wurth_Elektronik_Passive_Capacitors_rev18b:WCAP-CSGP_0402
- removed C25, C28: 18pF, rcl:C0603
- removed C30: CBEC219-3479B001C1AF, wouter:BTB_CONN_68_F
- removed C39: C3216X7R1H225K160AE, samacsys:CAPC3216X180N
- removed C40, C43, C44, C47: 1206 x7r 47uF 25V, samacsys:CAPC6050X550N
- removed C41, C42: 0.1uF x7r 1206, samacsys:CAPC3416X90N
- removed C45, C46: 1206 x7r 2.2uF 25V, rcl:C1206
- removed C77, C78, C79, C80, C81, C82, C83, C84: 100n, rcl:C050-025X075
- removed D0_0, D0_1, D1_0, D1_1, D2_0, D2_1, D3_0, D3_1, D4_0, D4_1, D5_0, D5_1, D6_0, D6_1, D7_0, D7_1: (no value), dfls130l-7:POWERDI-123
- removed D1, D2: BAT64-04E6433, BAT64-04E6433:SOT95P260X110-3N
- removed D10, D11, D12, D5, D6, D7, D8, D9: sbr3u20sa, dfls130l-7:POWERDI-123
- removed D13, D14, D17, D18, D19, D20, D3, D4: SBR1U200P1, dfls130l-7:POWERDI-123
- removed D15, D16, D21, D22: SBR3U20SA, dfls130l-7:POWERDI-123
- removed D25: MBRS360T3G, samacsys:DIOM7958X256N
- removed D26: VS-MBRS340-M3_9AT, samacsys:DIOM7959X262N
- removed GAIN12_1, GAIN34_1: 3361S-1-104GLF, 3361S-1-104GLF:3361S
- removed GND_1, TP2_10, TP2_11, TP2_12, TP2_5, TP2_6, TP2_7, TP2_8, TP2_9, TP2_GND1: 5019, 5019:TP380X203
- removed HVM$1, HVM_CW$1, HVP$1, HVP_CW$1, LVOUT_0, LVOUT_1, LVOUT_2, LVOUT_3, LVOUT_4, LVOUT_5, LVOUT_6, LVOUT_7, VDDM$1, VDDP$1: R141426, con-coax:R141426
- removed IC1: AD8334ACPZ, AD8334ACPZ:QFN50P900X900X100-65N
- removed IC3: LT8471EFE#PBF, samacsys:SOP65P640X120-21N
- removed IN0_0, IN0_1, LVOUT0, T_OUT_0, T_OUT_1, T_OUT_2, T_OUT_3, T_OUT_4, T_OUT_5, T_OUT_6, T_OUT_7: 5015, keystone_5015:KEYSTONE_5015
- removed J1: FMC-LPC, wouter:FMC-LPC-MALE
- removed JP1, JP2: (no value), jumper:JP1
- removed L1, L6: BLM21AG121SN1D, rcl:L2012C
- removed L2: 744025150, samacsys:WE-TPC_282892
- removed L27, L28, L29, L30, L31, L32: BLM21AG121SN1D, resistor:L2012C
- removed L7: 74437324068, samacsys:WE-LHMI_402048
- removed L8: 74437324100, samacsys:WE-LHMI_402048
- removed PGND+: GND, wirepad:3,17/1,3
- removed PGND-, PGNDD, PHVM, PHVM_CW, PHVP, PHVP_CW, PVDDM, PVDDP: (no value), wirepad:3,17/1,3
- removed POWER_BOARD_CONN: 43045-0809, con-molex-micro-fit-3_0:43045-0809
- removed R1, R3: 400k, resistor:R0603
- removed R17: 261k 25V, resistor:M1206
- removed R18: 82k 25V, resistor:M1206
- removed R19, R21: 316k, rcl:R1206
- removed R2: 10k, rcl:R0805
- removed R20, R22: 59k, rcl:R1206
- removed R23, R24: 100k, rcl:R1206
- removed R25: 187k, rcl:R1206
- removed R4, R5: 4.02k, resistor:R0805
- removed R43, R44, R45, R46, R47, R48, R49, R50: 1K, rcl:0207/7
- removed R6, R7: 274, resistor:R0603
- removed SLIDESWITCH1, SLIDESWITCH2: CL-SB-12A-01, wouter:CL-SB-12A-01
- removed SLIDESWITCH10, SLIDESWITCH11, SLIDESWITCH7, SLIDESWITCH9: CL-SB-22A-01, wouter:CL-SB-22A-01
- removed STHV_0: STHV800, wouter:TFLGA-56LD
- removed X10, X11, X12, X2, X3, X4, X5, X9: (no value), con-phoenix-254:2POL254
- added CONN_FPGA1:C30: CBEC219-3479B001C1AF, wouter:BTB_CONN_68_F
- added CONN_FPGA1:D13, CONN_FPGA1:D14, CONN_FPGA1:D17, CONN_FPGA1:D18, CONN_FPGA1:D19, CONN_FPGA1:D20, CONN_FPGA1:D3, CONN_FPGA1:D4: SBR1U200P1, dfls130l-7:POWERDI-123
- added CONN_FPGA1:D15, CONN_FPGA1:D16, CONN_FPGA1:D21, CONN_FPGA1:D22: SBR3U20SA, dfls130l-7:POWERDI-123
- added CONN_FPGA1:HVM$1, CONN_FPGA1:HVM_CW$1, CONN_FPGA1:HVP$1, CONN_FPGA1:HVP_CW$1, CONN_FPGA1:VDDM$1, CONN_FPGA1:VDDP$1: R141426, con-coax:R141426
- added CONN_FPGA1:J1: FMC-LPC, wouter:FMC-LPC-MALE
- added CONN_FPGA1:PGND+: GND, wirepad:3,17/1,3
- added CONN_FPGA1:PGND-, CONN_FPGA1:PGNDD, CONN_FPGA1:PHVM, CONN_FPGA1:PHVM_CW, CONN_FPGA1:PHVP, CONN_FPGA1:PHVP_CW, CONN_FPGA1:PVDDM, CONN_FPGA1:PVDDP: (no value), wirepad:3,17/1,3
- added CONN_FPGA1:POWER_BOARD_CONN: 43045-0809, con-molex-micro-fit-3_0:43045-0809
- added DRIVER1:C170, DRIVER1:C171, DRIVER1:C172, DRIVER1:C173, DRIVER1:C174, DRIVER1:C175, DRIVER1:C176, DRIVER1:C177, DRIVER1:C178, DRIVER1:C179, DRIVER1:C180, DRIVER1:C181, DRIVER1:C182, DRIVER1:C183, DRIVER1:C184, DRIVER1:C185, DRIVER1:C186, DRIVER1:C187, DRIVER1:C188, DRIVER1:C189, DRIVER1:C190, DRIVER1:C191, DRIVER2:C170, DRIVER2:C171, DRIVER2:C172, DRIVER2:C173, DRIVER2:C174, DRIVER2:C175, DRIVER2:C176, DRIVER2:C177, DRIVER2:C178, DRIVER2:C179, DRIVER2:C180, DRIVER2:C181, DRIVER2:C182, DRIVER2:C183, DRIVER2:C184, DRIVER2:C185, DRIVER2:C186, DRIVER2:C187, DRIVER2:C188, DRIVER2:C189, DRIVER2:C190, DRIVER2:C191: 220n 100V, rcl:C0805
- added DRIVER1:D0_0, DRIVER1:D0_1, DRIVER1:D1_0, DRIVER1:D1_1, DRIVER1:D2_0, DRIVER1:D2_1, DRIVER1:D3_0, DRIVER1:D3_1, DRIVER1:D4_0, DRIVER1:D4_1, DRIVER1:D5_0, DRIVER1:D5_1, DRIVER1:D6_0, DRIVER1:D6_1, DRIVER1:D7_0, DRIVER1:D7_1, DRIVER2:D0_0, DRIVER2:D0_1, DRIVER2:D1_0, DRIVER2:D1_1, DRIVER2:D2_0, DRIVER2:D2_1, DRIVER2:D3_0, DRIVER2:D3_1, DRIVER2:D4_0, DRIVER2:D4_1, DRIVER2:D5_0, DRIVER2:D5_1, DRIVER2:D6_0, DRIVER2:D6_1, DRIVER2:D7_0, DRIVER2:D7_1: (no value), dfls130l-7:POWERDI-123
- added DRIVER1:GND_1, DRIVER2:GND_1, RECEIVER1:S1:TP2_10, RECEIVER1:S1:TP2_11, RECEIVER1:S1:TP2_12, RECEIVER1:S1:TP2_5, RECEIVER1:S1:TP2_6, RECEIVER1:S1:TP2_7, RECEIVER1:S1:TP2_8, RECEIVER1:S1:TP2_9, RECEIVER1:S1:TP2_GND1, RECEIVER1:S2:TP2_10, RECEIVER1:S2:TP2_11, RECEIVER1:S2:TP2_12, RECEIVER1:S2:TP2_5, RECEIVER1:S2:TP2_6, RECEIVER1:S2:TP2_7, RECEIVER1:S2:TP2_8, RECEIVER1:S2:TP2_9, RECEIVER1:S2:TP2_GND1, RECEIVER2:S1:TP2_10, RECEIVER2:S1:TP2_11, RECEIVER2:S1:TP2_12, RECEIVER2:S1:TP2_5, RECEIVER2:S1:TP2_6, RECEIVER2:S1:TP2_7, RECEIVER2:S1:TP2_8, RECEIVER2:S1:TP2_9, RECEIVER2:S1:TP2_GND1, RECEIVER2:S2:TP2_10, RECEIVER2:S2:TP2_11, RECEIVER2:S2:TP2_12, RECEIVER2:S2:TP2_5, RECEIVER2:S2:TP2_6, RECEIVER2:S2:TP2_7, RECEIVER2:S2:TP2_8, RECEIVER2:S2:TP2_9, RECEIVER2:S2:TP2_GND1, RECEIVER3:S1:TP2_10, RECEIVER3:S1:TP2_11, RECEIVER3:S1:TP2_12, RECEIVER3:S1:TP2_5, RECEIVER3:S1:TP2_6, RECEIVER3:S1:TP2_7, RECEIVER3:S1:TP2_8, RECEIVER3:S1:TP2_9, RECEIVER3:S1:TP2_GND1, RECEIVER3:S2:TP2_10, RECEIVER3:S2:TP2_11, RECEIVER3:S2:TP2_12, RECEIVER3:S2:TP2_5, RECEIVER3:S2:TP2_6, RECEIVER3:S2:TP2_7, RECEIVER3:S2:TP2_8, RECEIVER3:S2:TP2_9, RECEIVER3:S2:TP2_GND1, RECEIVER4:S1:TP2_10, RECEIVER4:S1:TP2_11, RECEIVER4:S1:TP2_12, RECEIVER4:S1:TP2_5, RECEIVER4:S1:TP2_6, RECEIVER4:S1:TP2_7, RECEIVER4:S1:TP2_8, RECEIVER4:S1:TP2_9, RECEIVER4:S1:TP2_GND1, RECEIVER4:S2:TP2_10, RECEIVER4:S2:TP2_11, RECEIVER4:S2:TP2_12, RECEIVER4:S2:TP2_5, RECEIVER4:S2:TP2_6, RECEIVER4:S2:TP2_7, RECEIVER4:S2:TP2_8, RECEIVER4:S2:TP2_9, RECEIVER4:S2:TP2_GND1: 5019, 5019:TP380X203
- added DRIVER1:IN0_0, DRIVER1:IN0_1, DRIVER1:LVOUT0, DRIVER1:T_OUT_0, DRIVER1:T_OUT_1, DRIVER1:T_OUT_2, DRIVER1:T_OUT_3, DRIVER1:T_OUT_4, DRIVER1:T_OUT_5, DRIVER1:T_OUT_6, DRIVER1:T_OUT_7, DRIVER2:IN0_0, DRIVER2:IN0_1, DRIVER2:LVOUT0, DRIVER2:T_OUT_0, DRIVER2:T_OUT_1, DRIVER2:T_OUT_2, DRIVER2:T_OUT_3, DRIVER2:T_OUT_4, DRIVER2:T_OUT_5, DRIVER2:T_OUT_6, DRIVER2:T_OUT_7: 5015, keystone_5015:KEYSTONE_5015
- added DRIVER1:R2, DRIVER2:R2: 10k, rcl:R0805
- added DRIVER1:STHV_0, DRIVER2:STHV_0: STHV800, wouter:TFLGA-56LD
- added POWER1:C39: C3216X7R1H225K160AE, samacsys:CAPC3216X180N
- added POWER1:C40, POWER1:C43, POWER1:C44, POWER1:C47: 1206 x7r 47uF 25V, samacsys:CAPC6050X550N
- added POWER1:C41, POWER1:C42: 0.1uF x7r 1206, samacsys:CAPC3416X90N
- added POWER1:C45, POWER1:C46: 1206 x7r 2.2uF 25V, rcl:C1206
- added POWER1:D25: MBRS360T3G, samacsys:DIOM7958X256N
- added POWER1:D26: VS-MBRS340-M3_9AT, samacsys:DIOM7959X262N
- added POWER1:IC3: LT8471EFE#PBF, samacsys:SOP65P640X120-21N
- added POWER1:L2: 744025150, samacsys:WE-TPC_282892
- added POWER1:L7: 74437324068, samacsys:WE-LHMI_402048
- added POWER1:L8: 74437324100, samacsys:WE-LHMI_402048
- added POWER1:R17: 261k 25V, resistor:M1206
- added POWER1:R18: 82k 25V, resistor:M1206
- added POWER1:R19, POWER1:R21: 316k, rcl:R1206
- added POWER1:R20, POWER1:R22: 59k, rcl:R1206
- added POWER1:R23, POWER1:R24: 100k, rcl:R1206
- added POWER1:R25: 187k, rcl:R1206
- added RECEIVER1:ADC2:ADC1, RECEIVER2:ADC2:ADC1, RECEIVER3:ADC2:ADC1, RECEIVER4:ADC2:ADC1: LTC2344-16, wouter:QFN32
- added RECEIVER1:ADC2:C139, RECEIVER1:ADC2:C142, RECEIVER1:ADC2:C143, RECEIVER2:ADC2:C139, RECEIVER2:ADC2:C142, RECEIVER2:ADC2:C143, RECEIVER3:ADC2:C139, RECEIVER3:ADC2:C142, RECEIVER3:ADC2:C143, RECEIVER4:ADC2:C139, RECEIVER4:ADC2:C142, RECEIVER4:ADC2:C143: 0.1uf, rcl:C0402
- added RECEIVER1:ADC2:C140, RECEIVER2:ADC2:C140, RECEIVER3:ADC2:C140, RECEIVER4:ADC2:C140: 47uf, rcl:C1210
- added RECEIVER1:ADC2:C141, RECEIVER2:ADC2:C141, RECEIVER3:ADC2:C141, RECEIVER4:ADC2:C141: 2.2uf, rcl:C0402
- added RECEIVER1:S12:C77, RECEIVER1:S12:C78, RECEIVER1:S5:C77, RECEIVER1:S5:C78, RECEIVER1:S6:C77, RECEIVER1:S6:C78, RECEIVER1:S7:C77, RECEIVER1:S7:C78, RECEIVER2:S12:C77, RECEIVER2:S12:C78, RECEIVER2:S5:C77, RECEIVER2:S5:C78, RECEIVER2:S6:C77, RECEIVER2:S6:C78, RECEIVER2:S7:C77, RECEIVER2:S7:C78, RECEIVER3:S12:C77, RECEIVER3:S12:C78, RECEIVER3:S5:C77, RECEIVER3:S5:C78, RECEIVER3:S6:C77, RECEIVER3:S6:C78, RECEIVER3:S7:C77, RECEIVER3:S7:C78, RECEIVER4:S12:C77, RECEIVER4:S12:C78, RECEIVER4:S5:C77, RECEIVER4:S5:C78, RECEIVER4:S6:C77, RECEIVER4:S6:C78, RECEIVER4:S7:C77, RECEIVER4:S7:C78: 100n, rcl:C050-025X075
- added RECEIVER1:S12:D5, RECEIVER1:S12:D6, RECEIVER1:S5:D5, RECEIVER1:S5:D6, RECEIVER1:S6:D5, RECEIVER1:S6:D6, RECEIVER1:S7:D5, RECEIVER1:S7:D6, RECEIVER2:S12:D5, RECEIVER2:S12:D6, RECEIVER2:S5:D5, RECEIVER2:S5:D6, RECEIVER2:S6:D5, RECEIVER2:S6:D6, RECEIVER2:S7:D5, RECEIVER2:S7:D6, RECEIVER3:S12:D5, RECEIVER3:S12:D6, RECEIVER3:S5:D5, RECEIVER3:S5:D6, RECEIVER3:S6:D5, RECEIVER3:S6:D6, RECEIVER3:S7:D5, RECEIVER3:S7:D6, RECEIVER4:S12:D5, RECEIVER4:S12:D6, RECEIVER4:S5:D5, RECEIVER4:S5:D6, RECEIVER4:S6:D5, RECEIVER4:S6:D6, RECEIVER4:S7:D5, RECEIVER4:S7:D6: sbr3u20sa, dfls130l-7:POWERDI-123
- added RECEIVER1:S12:R43, RECEIVER1:S12:R44, RECEIVER1:S5:R43, RECEIVER1:S5:R44, RECEIVER1:S6:R43, RECEIVER1:S6:R44, RECEIVER1:S7:R43, RECEIVER1:S7:R44, RECEIVER2:S12:R43, RECEIVER2:S12:R44, RECEIVER2:S5:R43, RECEIVER2:S5:R44, RECEIVER2:S6:R43, RECEIVER2:S6:R44, RECEIVER2:S7:R43, RECEIVER2:S7:R44, RECEIVER3:S12:R43, RECEIVER3:S12:R44, RECEIVER3:S5:R43, RECEIVER3:S5:R44, RECEIVER3:S6:R43, RECEIVER3:S6:R44, RECEIVER3:S7:R43, RECEIVER3:S7:R44, RECEIVER4:S12:R43, RECEIVER4:S12:R44, RECEIVER4:S5:R43, RECEIVER4:S5:R44, RECEIVER4:S6:R43, RECEIVER4:S6:R44, RECEIVER4:S7:R43, RECEIVER4:S7:R44: 1K, rcl:0207/7
- added RECEIVER1:S12:SLIDESWITCH7, RECEIVER1:S5:SLIDESWITCH7, RECEIVER1:S6:SLIDESWITCH7, RECEIVER1:S7:SLIDESWITCH7, RECEIVER2:S12:SLIDESWITCH7, RECEIVER2:S5:SLIDESWITCH7, RECEIVER2:S6:SLIDESWITCH7, RECEIVER2:S7:SLIDESWITCH7, RECEIVER3:S12:SLIDESWITCH7, RECEIVER3:S5:SLIDESWITCH7, RECEIVER3:S6:SLIDESWITCH7, RECEIVER3:S7:SLIDESWITCH7, RECEIVER4:S12:SLIDESWITCH7, RECEIVER4:S5:SLIDESWITCH7, RECEIVER4:S6:SLIDESWITCH7, RECEIVER4:S7:SLIDESWITCH7: CL-SB-22A-01, wouter:CL-SB-22A-01
- added RECEIVER1:S12:X12, RECEIVER1:S12:X2, RECEIVER1:S5:X12, RECEIVER1:S5:X2, RECEIVER1:S6:X12, RECEIVER1:S6:X2, RECEIVER1:S7:X12, RECEIVER1:S7:X2, RECEIVER2:S12:X12, RECEIVER2:S12:X2, RECEIVER2:S5:X12, RECEIVER2:S5:X2, RECEIVER2:S6:X12, RECEIVER2:S6:X2, RECEIVER2:S7:X12, RECEIVER2:S7:X2, RECEIVER3:S12:X12, RECEIVER3:S12:X2, RECEIVER3:S5:X12, RECEIVER3:S5:X2, RECEIVER3:S6:X12, RECEIVER3:S6:X2, RECEIVER3:S7:X12, RECEIVER3:S7:X2, RECEIVER4:S12:X12, RECEIVER4:S12:X2, RECEIVER4:S5:X12, RECEIVER4:S5:X2, RECEIVER4:S6:X12, RECEIVER4:S6:X2, RECEIVER4:S7:X12, RECEIVER4:S7:X2: (no value), con-phoenix-254:2POL254
- added RECEIVER1:S1:C1, RECEIVER1:S1:C10, RECEIVER1:S1:C13, RECEIVER1:S1:C14, RECEIVER1:S1:C15, RECEIVER1:S1:C16, RECEIVER1:S1:C17, RECEIVER1:S1:C18, RECEIVER1:S1:C2, RECEIVER1:S1:C21, RECEIVER1:S1:C22, RECEIVER1:S1:C23, RECEIVER1:S1:C26, RECEIVER1:S1:C3, RECEIVER1:S1:C4, RECEIVER1:S1:C5, RECEIVER1:S1:C51, RECEIVER1:S1:C52, RECEIVER1:S1:C53, RECEIVER1:S1:C54, RECEIVER1:S1:C55, RECEIVER1:S1:C56, RECEIVER1:S1:C6, RECEIVER1:S1:C7, RECEIVER1:S1:C8, RECEIVER1:S1:C9, RECEIVER1:S2:C1, RECEIVER1:S2:C10, RECEIVER1:S2:C13, RECEIVER1:S2:C14, RECEIVER1:S2:C15, RECEIVER1:S2:C16, RECEIVER1:S2:C17, RECEIVER1:S2:C18, RECEIVER1:S2:C2, RECEIVER1:S2:C21, RECEIVER1:S2:C22, RECEIVER1:S2:C23, RECEIVER1:S2:C26, RECEIVER1:S2:C3, RECEIVER1:S2:C4, RECEIVER1:S2:C5, RECEIVER1:S2:C51, RECEIVER1:S2:C52, RECEIVER1:S2:C53, RECEIVER1:S2:C54, RECEIVER1:S2:C55, RECEIVER1:S2:C56, RECEIVER1:S2:C6, RECEIVER1:S2:C7, RECEIVER1:S2:C8, RECEIVER1:S2:C9, RECEIVER2:S1:C1, RECEIVER2:S1:C10, RECEIVER2:S1:C13, RECEIVER2:S1:C14, RECEIVER2:S1:C15, RECEIVER2:S1:C16, RECEIVER2:S1:C17, RECEIVER2:S1:C18, RECEIVER2:S1:C2, RECEIVER2:S1:C21, RECEIVER2:S1:C22, RECEIVER2:S1:C23, RECEIVER2:S1:C26, RECEIVER2:S1:C3, RECEIVER2:S1:C4, RECEIVER2:S1:C5, RECEIVER2:S1:C51, RECEIVER2:S1:C52, RECEIVER2:S1:C53, RECEIVER2:S1:C54, RECEIVER2:S1:C55, RECEIVER2:S1:C56, RECEIVER2:S1:C6, RECEIVER2:S1:C7, RECEIVER2:S1:C8, RECEIVER2:S1:C9, RECEIVER2:S2:C1, RECEIVER2:S2:C10, RECEIVER2:S2:C13, RECEIVER2:S2:C14, RECEIVER2:S2:C15, RECEIVER2:S2:C16, RECEIVER2:S2:C17, RECEIVER2:S2:C18, RECEIVER2:S2:C2, RECEIVER2:S2:C21, RECEIVER2:S2:C22, RECEIVER2:S2:C23, RECEIVER2:S2:C26, RECEIVER2:S2:C3, RECEIVER2:S2:C4, RECEIVER2:S2:C5, RECEIVER2:S2:C51, RECEIVER2:S2:C52, RECEIVER2:S2:C53, RECEIVER2:S2:C54, RECEIVER2:S2:C55, RECEIVER2:S2:C56, RECEIVER2:S2:C6, RECEIVER2:S2:C7, RECEIVER2:S2:C8, RECEIVER2:S2:C9, RECEIVER3:S1:C1, RECEIVER3:S1:C10, RECEIVER3:S1:C13, RECEIVER3:S1:C14, RECEIVER3:S1:C15, RECEIVER3:S1:C16, RECEIVER3:S1:C17, RECEIVER3:S1:C18, RECEIVER3:S1:C2, RECEIVER3:S1:C21, RECEIVER3:S1:C22, RECEIVER3:S1:C23, RECEIVER3:S1:C26, RECEIVER3:S1:C3, RECEIVER3:S1:C4, RECEIVER3:S1:C5, RECEIVER3:S1:C51, RECEIVER3:S1:C52, RECEIVER3:S1:C53, RECEIVER3:S1:C54, RECEIVER3:S1:C55, RECEIVER3:S1:C56, RECEIVER3:S1:C6, RECEIVER3:S1:C7, RECEIVER3:S1:C8, RECEIVER3:S1:C9, RECEIVER3:S2:C1, RECEIVER3:S2:C10, RECEIVER3:S2:C13, RECEIVER3:S2:C14, RECEIVER3:S2:C15, RECEIVER3:S2:C16, RECEIVER3:S2:C17, RECEIVER3:S2:C18, RECEIVER3:S2:C2, RECEIVER3:S2:C21, RECEIVER3:S2:C22, RECEIVER3:S2:C23, RECEIVER3:S2:C26, RECEIVER3:S2:C3, RECEIVER3:S2:C4, RECEIVER3:S2:C5, RECEIVER3:S2:C51, RECEIVER3:S2:C52, RECEIVER3:S2:C53, RECEIVER3:S2:C54, RECEIVER3:S2:C55, RECEIVER3:S2:C56, RECEIVER3:S2:C6, RECEIVER3:S2:C7, RECEIVER3:S2:C8, RECEIVER3:S2:C9, RECEIVER4:S1:C1, RECEIVER4:S1:C10, RECEIVER4:S1:C13, RECEIVER4:S1:C14, RECEIVER4:S1:C15, RECEIVER4:S1:C16, RECEIVER4:S1:C17, RECEIVER4:S1:C18, RECEIVER4:S1:C2, RECEIVER4:S1:C21, RECEIVER4:S1:C22, RECEIVER4:S1:C23, RECEIVER4:S1:C26, RECEIVER4:S1:C3, RECEIVER4:S1:C4, RECEIVER4:S1:C5, RECEIVER4:S1:C51, RECEIVER4:S1:C52, RECEIVER4:S1:C53, RECEIVER4:S1:C54, RECEIVER4:S1:C55, RECEIVER4:S1:C56, RECEIVER4:S1:C6, RECEIVER4:S1:C7, RECEIVER4:S1:C8, RECEIVER4:S1:C9, RECEIVER4:S2:C1, RECEIVER4:S2:C10, RECEIVER4:S2:C13, RECEIVER4:S2:C14, RECEIVER4:S2:C15, RECEIVER4:S2:C16, RECEIVER4:S2:C17, RECEIVER4:S2:C18, RECEIVER4:S2:C2, RECEIVER4:S2:C21, RECEIVER4:S2:C22, RECEIVER4:S2:C23, RECEIVER4:S2:C26, RECEIVER4:S2:C3, RECEIVER4:S2:C4, RECEIVER4:S2:C5, RECEIVER4:S2:C51, RECEIVER4:S2:C52, RECEIVER4:S2:C53, RECEIVER4:S2:C54, RECEIVER4:S2:C55, RECEIVER4:S2:C56, RECEIVER4:S2:C6, RECEIVER4:S2:C7, RECEIVER4:S2:C8, RECEIVER4:S2:C9: 0.1uF, Wurth_Elektronik_Passive_Capacitors_rev18b:WCAP-CSGP_0402
- added RECEIVER1:S1:C19, RECEIVER1:S1:C20, RECEIVER1:S2:C19, RECEIVER1:S2:C20, RECEIVER2:S1:C19, RECEIVER2:S1:C20, RECEIVER2:S2:C19, RECEIVER2:S2:C20, RECEIVER3:S1:C19, RECEIVER3:S1:C20, RECEIVER3:S2:C19, RECEIVER3:S2:C20, RECEIVER4:S1:C19, RECEIVER4:S1:C20, RECEIVER4:S2:C19, RECEIVER4:S2:C20: 1nF, rcl:C0402
- added RECEIVER1:S1:C24, RECEIVER1:S1:C27, RECEIVER1:S2:C24, RECEIVER1:S2:C27, RECEIVER2:S1:C24, RECEIVER2:S1:C27, RECEIVER2:S2:C24, RECEIVER2:S2:C27, RECEIVER3:S1:C24, RECEIVER3:S1:C27, RECEIVER3:S2:C24, RECEIVER3:S2:C27, RECEIVER4:S1:C24, RECEIVER4:S1:C27, RECEIVER4:S2:C24, RECEIVER4:S2:C27: 22pF, Wurth_Elektronik_Passive_Capacitors_rev18b:WCAP-CSGP_0402
- added RECEIVER1:S1:C25, RECEIVER1:S1:C28, RECEIVER1:S2:C25, RECEIVER1:S2:C28, RECEIVER2:S1:C25, RECEIVER2:S1:C28, RECEIVER2:S2:C25, RECEIVER2:S2:C28, RECEIVER3:S1:C25, RECEIVER3:S1:C28, RECEIVER3:S2:C25, RECEIVER3:S2:C28, RECEIVER4:S1:C25, RECEIVER4:S1:C28, RECEIVER4:S2:C25, RECEIVER4:S2:C28: 18nF, rcl:C0603
- added RECEIVER1:S1:D1, RECEIVER1:S1:D2, RECEIVER1:S2:D1, RECEIVER1:S2:D2, RECEIVER2:S1:D1, RECEIVER2:S1:D2, RECEIVER2:S2:D1, RECEIVER2:S2:D2, RECEIVER3:S1:D1, RECEIVER3:S1:D2, RECEIVER3:S2:D1, RECEIVER3:S2:D2, RECEIVER4:S1:D1, RECEIVER4:S1:D2, RECEIVER4:S2:D1, RECEIVER4:S2:D2: BAT64-04E6433, BAT64-04E6433:SOT95P260X110-3N
- added RECEIVER1:S1:GAIN12_1, RECEIVER1:S1:GAIN34_1, RECEIVER1:S2:GAIN12_1, RECEIVER1:S2:GAIN34_1, RECEIVER2:S1:GAIN12_1, RECEIVER2:S1:GAIN34_1, RECEIVER2:S2:GAIN12_1, RECEIVER2:S2:GAIN34_1, RECEIVER3:S1:GAIN12_1, RECEIVER3:S1:GAIN34_1, RECEIVER3:S2:GAIN12_1, RECEIVER3:S2:GAIN34_1, RECEIVER4:S1:GAIN12_1, RECEIVER4:S1:GAIN34_1, RECEIVER4:S2:GAIN12_1, RECEIVER4:S2:GAIN34_1: 3361S-1-104GLF, 3361S-1-104GLF:3361S
- added RECEIVER1:S1:IC1, RECEIVER1:S2:IC1, RECEIVER2:S1:IC1, RECEIVER2:S2:IC1, RECEIVER3:S1:IC1, RECEIVER3:S2:IC1, RECEIVER4:S1:IC1, RECEIVER4:S2:IC1: AD8334ACPZ, AD8334ACPZ:QFN50P900X900X100-65N
- added RECEIVER1:S1:JP1, RECEIVER1:S1:JP2, RECEIVER1:S2:JP1, RECEIVER1:S2:JP2, RECEIVER2:S1:JP1, RECEIVER2:S1:JP2, RECEIVER2:S2:JP1, RECEIVER2:S2:JP2, RECEIVER3:S1:JP1, RECEIVER3:S1:JP2, RECEIVER3:S2:JP1, RECEIVER3:S2:JP2, RECEIVER4:S1:JP1, RECEIVER4:S1:JP2, RECEIVER4:S2:JP1, RECEIVER4:S2:JP2: (no value), jumper:JP1
- added RECEIVER1:S1:L1, RECEIVER1:S1:L6, RECEIVER1:S2:L1, RECEIVER1:S2:L6, RECEIVER2:S1:L1, RECEIVER2:S1:L6, RECEIVER2:S2:L1, RECEIVER2:S2:L6, RECEIVER3:S1:L1, RECEIVER3:S1:L6, RECEIVER3:S2:L1, RECEIVER3:S2:L6, RECEIVER4:S1:L1, RECEIVER4:S1:L6, RECEIVER4:S2:L1, RECEIVER4:S2:L6: BLM21AG121SN1D, rcl:L2012C
- added RECEIVER1:S1:L27, RECEIVER1:S1:L28, RECEIVER1:S1:L29, RECEIVER1:S1:L30, RECEIVER1:S1:L31, RECEIVER1:S1:L32, RECEIVER1:S2:L27, RECEIVER1:S2:L28, RECEIVER1:S2:L29, RECEIVER1:S2:L30, RECEIVER1:S2:L31, RECEIVER1:S2:L32, RECEIVER2:S1:L27, RECEIVER2:S1:L28, RECEIVER2:S1:L29, RECEIVER2:S1:L30, RECEIVER2:S1:L31, RECEIVER2:S1:L32, RECEIVER2:S2:L27, RECEIVER2:S2:L28, RECEIVER2:S2:L29, RECEIVER2:S2:L30, RECEIVER2:S2:L31, RECEIVER2:S2:L32, RECEIVER3:S1:L27, RECEIVER3:S1:L28, RECEIVER3:S1:L29, RECEIVER3:S1:L30, RECEIVER3:S1:L31, RECEIVER3:S1:L32, RECEIVER3:S2:L27, RECEIVER3:S2:L28, RECEIVER3:S2:L29, RECEIVER3:S2:L30, RECEIVER3:S2:L31, RECEIVER3:S2:L32, RECEIVER4:S1:L27, RECEIVER4:S1:L28, RECEIVER4:S1:L29, RECEIVER4:S1:L30, RECEIVER4:S1:L31, RECEIVER4:S1:L32, RECEIVER4:S2:L27, RECEIVER4:S2:L28, RECEIVER4:S2:L29, RECEIVER4:S2:L30, RECEIVER4:S2:L31, RECEIVER4:S2:L32: BLM21AG121SN1D, resistor:L2012C
- added RECEIVER1:S1:R1, RECEIVER1:S1:R3, RECEIVER1:S2:R1, RECEIVER1:S2:R3, RECEIVER2:S1:R1, RECEIVER2:S1:R3, RECEIVER2:S2:R1, RECEIVER2:S2:R3, RECEIVER3:S1:R1, RECEIVER3:S1:R3, RECEIVER3:S2:R1, RECEIVER3:S2:R3, RECEIVER4:S1:R1, RECEIVER4:S1:R3, RECEIVER4:S2:R1, RECEIVER4:S2:R3: 400k, resistor:R0603
- added RECEIVER1:S1:R4, RECEIVER1:S1:R5, RECEIVER1:S2:R4, RECEIVER1:S2:R5, RECEIVER2:S1:R4, RECEIVER2:S1:R5, RECEIVER2:S2:R4, RECEIVER2:S2:R5, RECEIVER3:S1:R4, RECEIVER3:S1:R5, RECEIVER3:S2:R4, RECEIVER3:S2:R5, RECEIVER4:S1:R4, RECEIVER4:S1:R5, RECEIVER4:S2:R4, RECEIVER4:S2:R5: 4.02k, resistor:R0805
- added RECEIVER1:S1:R6, RECEIVER1:S1:R7, RECEIVER1:S2:R6, RECEIVER1:S2:R7, RECEIVER2:S1:R6, RECEIVER2:S1:R7, RECEIVER2:S2:R6, RECEIVER2:S2:R7, RECEIVER3:S1:R6, RECEIVER3:S1:R7, RECEIVER3:S2:R6, RECEIVER3:S2:R7, RECEIVER4:S1:R6, RECEIVER4:S1:R7, RECEIVER4:S2:R6, RECEIVER4:S2:R7: 274, resistor:R0603
- added RECEIVER1:S1:R8, RECEIVER1:S1:R9, RECEIVER1:S2:R8, RECEIVER1:S2:R9, RECEIVER2:S1:R8, RECEIVER2:S1:R9, RECEIVER2:S2:R8, RECEIVER2:S2:R9, RECEIVER3:S1:R8, RECEIVER3:S1:R9, RECEIVER3:S2:R8, RECEIVER3:S2:R9, RECEIVER4:S1:R8, RECEIVER4:S1:R9, RECEIVER4:S2:R8, RECEIVER4:S2:R9: 0R, resistor:R0603
- added RECEIVER1:S1:SLIDESWITCH1, RECEIVER1:S1:SLIDESWITCH2, RECEIVER1:S2:SLIDESWITCH1, RECEIVER1:S2:SLIDESWITCH2, RECEIVER2:S1:SLIDESWITCH1, RECEIVER2:S1:SLIDESWITCH2, RECEIVER2:S2:SLIDESWITCH1, RECEIVER2:S2:SLIDESWITCH2, RECEIVER3:S1:SLIDESWITCH1, RECEIVER3:S1:SLIDESWITCH2, RECEIVER3:S2:SLIDESWITCH1, RECEIVER3:S2:SLIDESWITCH2, RECEIVER4:S1:SLIDESWITCH1, RECEIVER4:S1:SLIDESWITCH2, RECEIVER4:S2:SLIDESWITCH1, RECEIVER4:S2:SLIDESWITCH2: CL-SB-12A-01, wouter:CL-SB-12A-01
Connections:
- removed net /CS: ADC1.27
- removed net 3P3V: J1.C39, J1.D40
- removed net 3V3: ADC1.21, C143.1
- removed net 5V: ADC1.30, C142.1, L27.1, L28.1, L29.1, L30.1, L31.1, L32.1, R1.2, R3.2, SLIDESWITCH1.P$3, SLIDESWITCH2.P$3
- removed net ADIN1_N: ADC1.7
- removed net ADIN1_P: ADC1.8
- removed net ADIN2_N: ADC1.5
- removed net ADIN2_P: ADC1.6
- removed net ADIN3_N: ADC1.3
- removed net ADIN3_P: ADC1.4
- removed net ADIN4_N: ADC1.1
- removed net ADIN4_P: ADC1.2
- removed net BUSY: ADC1.26
- removed net C3: IC3.13, L2.1
- removed net CLAMP12_1: C22.1, IC1.53, JP1.1
- removed net CLAMP12_2: C21.1, IC1.28, JP2.1
- removed net CLK: STHV_0.CK
- removed net CNV: ADC1.15
- removed net CW: STHV_0.CW
- removed net DVDD: C182.1, R2.2, STHV_0.DVDD
- removed net E1: D26.1, IC3.2, L7.1
- removed net E2: D25.1, IC3.19, L8.2
- removed net EN12: IC1.52
- removed net EN34: IC1.51
- removed net ENV1_N: C78.1, D6.A, R44.2, X12.2
- removed net ENV1_P: C77.1, D5.C, R43.2, X12.1
- removed net ENV2_N: C80.1, D8.A, R46.2, X11.2
- removed net ENV2_P: C79.1, D7.C, R45.2, X11.1
- removed net ENV3_N: C82.1, D10.A, R48.2, X9.2
- removed net ENV3_P: C81.1, D9.C, R47.2, X9.1
- removed net ENV4_N: C84.1, D12.A, R50.2, X10.2
- removed net ENV4_P: C83.1, D11.C, R49.2, X10.1
- removed net FB1: IC3.5, R19.1, R20.2
- removed net FB2: IC3.16, R21.1, R22.2
- removed net GAIN12_1: C20.1, GAIN12_1.3, IC1.54, R3.1
- removed net GAIN12_2: C19.1, GAIN34_1.3, IC1.27, R1.1
- removed net GND: ADC1.11, ADC1.13, ADC1.14, ADC1.20, ADC1.29, ADC1.31, ADC1.32, ADC1.9, ADC1.EXP, C10.1, C139.2, C140.2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
- removed net HILO_12: IC1.29, SLIDESWITCH2.P$2
- removed net HVM: C183.1, C184.1, C185.1, C186.1, C187.1, C188.1, D0_1.A, D18.A, D1_1.A, D2_1.A, D3_1.A, D4.A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
- removed net HVM_CW: C189.2, C190.2, C191.2, D17.A, D3.A, POWER_BOARD_CONN.P$6, STHV_0.HVM_CW
- removed net HVP: C171.1, C172.1, C173.1, C174.1, C175.1, C176.1, D0_0.C, D13.C, D19.C, D1_0.C, D2_0.C, D3_0.C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
- removed net HVP_CW: C177.2, C178.2, C179.2, C40.2, C45.1, C46.2, D14.C, D20.C, IC3.1, IC3.20, L2.2, POWER_BOARD_CONN.P$2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
- removed net IN0_0: J1.G6, STHV_0.IN1_0
- removed net IN0_1: J1.G7, STHV_0.IN1_1
- removed net IN10_0: J1.G21
- removed net IN10_1: J1.G22
- removed net IN11_0: J1.H22
- removed net IN11_1: J1.H23
- removed net IN12_0: J1.G24
- removed net IN12_1: J1.G25
- removed net IN13_0: J1.H25
- removed net IN13_1: J1.H26
- removed net IN14_0: J1.G27
- removed net IN14_1: J1.G28
- removed net IN15_0: J1.H28
- removed net IN15_1: J1.H29
- removed net IN1_0: J1.H7, STHV_0.IN2_0
- removed net IN1_1: J1.H8, STHV_0.IN2_1
- removed net IN2_0: J1.G9, STHV_0.IN3_0
- removed net IN2_1: J1.G10, STHV_0.IN3_1
- removed net IN3_0: J1.H10, STHV_0.IN4_0
- removed net IN3_1: J1.H11, STHV_0.IN4_1
- removed net IN4_0: J1.G12, STHV_0.IN5_0
- removed net IN4_1: J1.G13, STHV_0.IN5_1
- removed net IN5_0: J1.H13, STHV_0.IN6_0
- removed net IN5_1: J1.H14, STHV_0.IN6_1
- removed net IN6_0: J1.G15, STHV_0.IN7_0
- removed net IN6_1: J1.G16, STHV_0.IN7_1
- removed net IN7_0: J1.H16, STHV_0.IN8_0
- removed net IN7_1: J1.H17, STHV_0.IN8_1
- removed net IN8_0: J1.G18
- removed net IN8_1: J1.G19
- removed net IN9_0: J1.H19
- removed net IN9_1: J1.H20
- removed net INH2: C23.1, C24.2, C25.1, IC1.1
- removed net INH4: C26.1, C27.2, C28.1, IC1.16
- removed net INX_1_0: IN0_1.1
- removed net LA28_N: J1.H32
- removed net LA28_P: J1.H31
- removed net LA30_N: J1.H35
- removed net LA30_P: J1.H34
- removed net LA32_N: J1.H38
- removed net LA32_P: J1.H37
- removed net LVOUT_0: D1.3, L1.1, LVOUT0.1, LVOUT_0.1, STHV_0.LVOUT_1
- removed net LVOUT_1: D2.3, L6.1, LVOUT_1.1, STHV_0.LVOUT_2
- removed net LVOUT_2: LVOUT_2.1, STHV_0.LVOUT_3
- removed net LVOUT_3: LVOUT_3.1, STHV_0.LVOUT_4
- removed net LVOUT_4: LVOUT_4.1, STHV_0.LVOUT_5
- removed net LVOUT_5: LVOUT_5.1, STHV_0.LVOUT_6
- removed net LVOUT_6: LVOUT_6.1, STHV_0.LVOUT_7
- removed net LVOUT_7: LVOUT_7.1, STHV_0.LVOUT_8
- removed net MODE_12: IC1.41, SLIDESWITCH1.P$2
- removed net N$1: C5.1, IC1.61
- removed net N$10: GAIN12_1.1
- removed net N$11: C23.2, L1.2
- removed net N$12: C25.2, R6.2
- removed net N$13: C26.2, L6.2
- removed net N$14: C28.2, R7.2
- removed net N$15: C12.1
- removed net N$17: D3.C, HVM_CW$1.1
- removed net N$18: D4.C, HVM$1.1
- removed net N$19: D13.A, HVP$1.1
- removed net N$2: C8.2, IC1.20
- removed net N$20: D14.A, HVP_CW$1.1
- removed net N$21: D15.A, VDDP$1.1
- removed net N$22: D16.C, VDDM$1.1
- removed net N$23: R2.1, STHV_0.THSD
- removed net N$24: C170.1, STHV_0.SUB
- removed net N$25: D19.A, PHVP.1
- removed net N$26: D20.A, PHVP_CW.1
- removed net N$27: D21.A, PVDDP.1
- removed net N$28: D22.C, PVDDM.1
- removed net N$3: D17.C, PHVM_CW.1
- removed net N$4: D18.C, PHVM.1
- removed net N$5: C10.2, IC1.2
- removed net N$6: C9.2, IC1.15
- removed net N$7: JP1.2, R4.1
- removed net N$8: JP2.2, R5.1
- removed net N$81: ADC1.10, C139.1
- removed net N$82: ADC1.12, C140.1
- removed net N$83: ADC1.28, C141.1
- removed net N$9: GAIN34_1.1
- removed net N5V: C44.2, D25.2, R21.2
- removed net OUT_0: C30.2, D0_0.A, D0_1.C, STHV_0.XDCR_1, T_OUT_0.1
- removed net OUT_1: C30.3, D1_0.A, D1_1.C, STHV_0.XDCR_2, T_OUT_1.1
- removed net OUT_10: C30.12
- removed net OUT_11: C30.13
- removed net OUT_12: C30.14
- removed net OUT_13: C30.15
- removed net OUT_14: C30.16
- removed net OUT_15: C30.17
- removed net OUT_16: C30.18
- removed net OUT_17: C30.19
- removed net OUT_18: C30.20
- removed net OUT_19: C30.21
- removed net OUT_2: C30.4, D2_0.A, D2_1.C, STHV_0.XDCR_3, T_OUT_2.1
- removed net OUT_20: C30.22
- removed net OUT_21: C30.23
- removed net OUT_22: C30.24
- removed net OUT_23: C30.25
- removed net OUT_24: C30.26
- removed net OUT_25: C30.27
- removed net OUT_26: C30.28
- removed net OUT_27: C30.29
- removed net OUT_28: C30.30
- removed net OUT_29: C30.31
- removed net OUT_3: C30.5, D3_0.A, D3_1.C, STHV_0.XDCR_4, T_OUT_3.1
- removed net OUT_30: C30.32
- removed net OUT_31: C30.33
- removed net OUT_32: C30.36
- removed net OUT_33: C30.37
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
Commit message: WIP Driver sheet
Connections:
- net RECEIVER1:ADC2:/CS renamed RECEIVER1:!CS
- net RECEIVER1:ADC2:BUSY renamed RECEIVER1:BUSY
- net RECEIVER1:ADC2:CNV renamed RECEIVER1:CNV
- net RECEIVER1:ADC2:SCKI renamed RECEIVER1:SCKI
- net RECEIVER1:ADC2:SDI renamed RECEIVER1:SDI
- net RECEIVER1:ADC2:SDO0 renamed RECEIVER1:SDO0
- net RECEIVER1:ADC2:SDO1 renamed RECEIVER1:SDO1
- net RECEIVER1:ADC2:SDO2 renamed RECEIVER1:SDO2
- net RECEIVER1:ADC2:SDO3 renamed RECEIVER1:SDO3
- net RECEIVER2:ADC2:/CS renamed RECEIVER2:!CS
- net RECEIVER2:ADC2:BUSY renamed RECEIVER2:BUSY
- net RECEIVER2:ADC2:CNV renamed RECEIVER2:CNV
- net RECEIVER2:ADC2:SCKI renamed RECEIVER2:SCKI
- net RECEIVER2:ADC2:SDI renamed RECEIVER2:SDI
- net RECEIVER2:ADC2:SDO0 renamed RECEIVER2:SDO0
- net RECEIVER2:ADC2:SDO1 renamed RECEIVER2:SDO1
- net RECEIVER2:ADC2:SDO2 renamed RECEIVER2:SDO2
- net RECEIVER2:ADC2:SDO3 renamed RECEIVER2:SDO3
- net RECEIVER3:ADC2:/CS renamed RECEIVER3:!CS
- net RECEIVER3:ADC2:BUSY renamed RECEIVER3:BUSY
- net RECEIVER3:ADC2:CNV renamed RECEIVER3:CNV
- net RECEIVER3:ADC2:SCKI renamed RECEIVER3:SCKI
- net RECEIVER3:ADC2:SDI renamed RECEIVER3:SDI
- net RECEIVER3:ADC2:SDO0 renamed RECEIVER3:SDO0
- net RECEIVER3:ADC2:SDO1 renamed RECEIVER3:SDO1
- net RECEIVER3:ADC2:SDO2 renamed RECEIVER3:SDO2
- net RECEIVER3:ADC2:SDO3 renamed RECEIVER3:SDO3
- net RECEIVER4:ADC2:/CS renamed RECEIVER4:!CS
- net RECEIVER4:ADC2:BUSY renamed RECEIVER4:BUSY
- net RECEIVER4:ADC2:CNV renamed RECEIVER4:CNV
- net RECEIVER4:ADC2:SCKI renamed RECEIVER4:SCKI
- net RECEIVER4:ADC2:SDI renamed RECEIVER4:SDI
- net RECEIVER4:ADC2:SDO0 renamed RECEIVER4:SDO0
- net RECEIVER4:ADC2:SDO1 renamed RECEIVER4:SDO1
- net RECEIVER4:ADC2:SDO2 renamed RECEIVER4:SDO2
- net RECEIVER4:ADC2:SDO3 renamed RECEIVER4:SDO3
- net DRIVER1:GND: now also DRIVER1:C171.1, DRIVER1:C172.1, DRIVER1:C173.1, DRIVER1:C174.1, DRIVER1:C175.1, DRIVER1:C176.1; no longer DRIVER1:C171.2, DRIVER1:C172.2, DRIVER1:C173.2, DRIVER1:C174.2, DRIVER1:C175.2, DRIVER1:C176.2
- net DRIVER1:HVP: now also DRIVER1:C171.2, DRIVER1:C172.2, DRIVER1:C173.2, DRIVER1:C174.2, DRIVER1:C175.2, DRIVER1:C176.2; no longer DRIVER1:C171.1, DRIVER1:C172.1, DRIVER1:C173.1, DRIVER1:C174.1, DRIVER1:C175.1, DRIVER1:C176.1
- net DRIVER2:GND: now also DRIVER2:C171.1, DRIVER2:C172.1, DRIVER2:C173.1, DRIVER2:C174.1, DRIVER2:C175.1, DRIVER2:C176.1; no longer DRIVER2:C171.2, DRIVER2:C172.2, DRIVER2:C173.2, DRIVER2:C174.2, DRIVER2:C175.2, DRIVER2:C176.2
- net DRIVER2:HVP: now also DRIVER2:C171.2, DRIVER2:C172.2, DRIVER2:C173.2, DRIVER2:C174.2, DRIVER2:C175.2, DRIVER2:C176.2; no longer DRIVER2:C171.1, DRIVER2:C172.1, DRIVER2:C173.1, DRIVER2:C174.1, DRIVER2:C175.1, DRIVER2:C176.1
