File: silense.brd (EAGLE design)
At the start: 160 x 100 mm, 854 parts

Commit message: main board: added all fpga connections
Connections:
- net CONN_FPGA1:LA28_P renamed CONN_FPGA1:CW
- net CONN_FPGA1:LA30_N renamed CONN_FPGA1:SDO0_2
- net CONN_FPGA1:LA30_P renamed CONN_FPGA1:SDO0_3
- net CONN_FPGA1:LA32_N renamed CONN_FPGA1:CNV1
- net CONN_FPGA1:LA32_P renamed CONN_FPGA1:CNV0
- removed net CONN_FPGA1:LA28_N: CONN_FPGA1:J1.H32
- new net CONN_FPGA1:ADC_CLK3: CONN_FPGA1:J1.G2
- new net CONN_FPGA1:ADC_CLK_0: CONN_FPGA1:J1.G6
- new net CONN_FPGA1:ADC_CLK_1: CONN_FPGA1:J1.G7
- new net CONN_FPGA1:ADC_CLK_2: CONN_FPGA1:J1.H4
- new net CONN_FPGA1:BUSY0: CONN_FPGA1:J1.D26
- new net CONN_FPGA1:BUSY1: CONN_FPGA1:J1.D27
- new net CONN_FPGA1:BUSY2: CONN_FPGA1:J1.C26
- new net CONN_FPGA1:BUSY3: CONN_FPGA1:J1.C27
- new net CONN_FPGA1:CNV2: CONN_FPGA1:J1.G36
- new net CONN_FPGA1:CNV3: CONN_FPGA1:J1.G37
- new net CONN_FPGA1:CS0: CONN_FPGA1:J1.D8
- new net CONN_FPGA1:CS1: CONN_FPGA1:J1.D9
- new net CONN_FPGA1:CS2: CONN_FPGA1:J1.C22
- new net CONN_FPGA1:CS3: CONN_FPGA1:J1.C23
- new net CONN_FPGA1:SDI0: CONN_FPGA1:J1.D20
- new net CONN_FPGA1:SDI1: CONN_FPGA1:J1.D21
- new net CONN_FPGA1:SDI2: CONN_FPGA1:J1.D23
- new net CONN_FPGA1:SDI3: CONN_FPGA1:J1.D24
- new net CONN_FPGA1:SDO0_0: CONN_FPGA1:J1.G34
- new net CONN_FPGA1:SDO0_1: CONN_FPGA1:J1.G33
- new net CONN_FPGA1:SDO1_0: CONN_FPGA1:J1.C11
- new net CONN_FPGA1:SDO1_1: CONN_FPGA1:J1.C10
- new net CONN_FPGA1:SDO1_2: CONN_FPGA1:J1.D12
- new net CONN_FPGA1:SDO1_3: CONN_FPGA1:J1.D11
- new net CONN_FPGA1:SDO2_0: CONN_FPGA1:J1.C15
- new net CONN_FPGA1:SDO2_1: CONN_FPGA1:J1.C14
- new net CONN_FPGA1:SDO2_2: CONN_FPGA1:J1.D15
- new net CONN_FPGA1:SDO2_3: CONN_FPGA1:J1.D14
- new net CONN_FPGA1:SDO3_0: CONN_FPGA1:J1.D18
- new net CONN_FPGA1:SDO3_1: CONN_FPGA1:J1.D17
- new net CONN_FPGA1:SDO3_2: CONN_FPGA1:J1.C19
- new net CONN_FPGA1:SDO3_3: CONN_FPGA1:J1.C18
- net CONN_FPGA1:IN0_0: now also CONN_FPGA1:J1.H7; no longer CONN_FPGA1:J1.G6
- net CONN_FPGA1:IN0_1: now also CONN_FPGA1:J1.H8; no longer CONN_FPGA1:J1.G7
- net CONN_FPGA1:IN10_0: now also CONN_FPGA1:J1.H22; no longer CONN_FPGA1:J1.G21
- net CONN_FPGA1:IN10_1: now also CONN_FPGA1:J1.H23; no longer CONN_FPGA1:J1.G22
- net CONN_FPGA1:IN11_0: now also CONN_FPGA1:J1.G24; no longer CONN_FPGA1:J1.H22
- net CONN_FPGA1:IN11_1: now also CONN_FPGA1:J1.G25; no longer CONN_FPGA1:J1.H23
- net CONN_FPGA1:IN12_0: now also CONN_FPGA1:J1.H25; no longer CONN_FPGA1:J1.G24
- net CONN_FPGA1:IN12_1: now also CONN_FPGA1:J1.H26; no longer CONN_FPGA1:J1.G25
- net CONN_FPGA1:IN13_0: now also CONN_FPGA1:J1.G27; no longer CONN_FPGA1:J1.H25
- net CONN_FPGA1:IN13_1: now also CONN_FPGA1:J1.G28; no longer CONN_FPGA1:J1.H26
- net CONN_FPGA1:IN14_0: now also CONN_FPGA1:J1.H28; no longer CONN_FPGA1:J1.G27
- net CONN_FPGA1:IN14_1: now also CONN_FPGA1:J1.H29; no longer CONN_FPGA1:J1.G28
- net CONN_FPGA1:IN15_0: now also CONN_FPGA1:J1.G30; no longer CONN_FPGA1:J1.H28
- net CONN_FPGA1:IN15_1: now also CONN_FPGA1:J1.G31; no longer CONN_FPGA1:J1.H29
- net CONN_FPGA1:IN1_0: now also CONN_FPGA1:J1.G9; no longer CONN_FPGA1:J1.H7
- net CONN_FPGA1:IN1_1: now also CONN_FPGA1:J1.G10; no longer CONN_FPGA1:J1.H8
- net CONN_FPGA1:IN2_0: now also CONN_FPGA1:J1.H10; no longer CONN_FPGA1:J1.G9
- net CONN_FPGA1:IN2_1: now also CONN_FPGA1:J1.H11; no longer CONN_FPGA1:J1.G10
- net CONN_FPGA1:IN3_0: now also CONN_FPGA1:J1.G12; no longer CONN_FPGA1:J1.H10
- net CONN_FPGA1:IN3_1: now also CONN_FPGA1:J1.G13; no longer CONN_FPGA1:J1.H11
- net CONN_FPGA1:IN4_0: now also CONN_FPGA1:J1.H13; no longer CONN_FPGA1:J1.G12
- net CONN_FPGA1:IN4_1: now also CONN_FPGA1:J1.H14; no longer CONN_FPGA1:J1.G13
- net CONN_FPGA1:IN5_0: now also CONN_FPGA1:J1.G15; no longer CONN_FPGA1:J1.H13
- net CONN_FPGA1:IN5_1: now also CONN_FPGA1:J1.G16; no longer CONN_FPGA1:J1.H14
- net CONN_FPGA1:IN6_0: now also CONN_FPGA1:J1.H16; no longer CONN_FPGA1:J1.G15
- net CONN_FPGA1:IN6_1: now also CONN_FPGA1:J1.H17; no longer CONN_FPGA1:J1.G16
- net CONN_FPGA1:IN7_0: now also CONN_FPGA1:J1.G18; no longer CONN_FPGA1:J1.H16
- net CONN_FPGA1:IN7_1: now also CONN_FPGA1:J1.G19; no longer CONN_FPGA1:J1.H17
- net CONN_FPGA1:IN8_0: now also CONN_FPGA1:J1.H19; no longer CONN_FPGA1:J1.G18
- net CONN_FPGA1:IN8_1: now also CONN_FPGA1:J1.H20; no longer CONN_FPGA1:J1.G19
- net CONN_FPGA1:IN9_0: now also CONN_FPGA1:J1.G21; no longer CONN_FPGA1:J1.H19
- net CONN_FPGA1:IN9_1: now also CONN_FPGA1:J1.G22; no longer CONN_FPGA1:J1.H20
Changed lines of the file:
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@@
 <?xml version="1.0" encoding="utf-8"?>
 <!DOCTYPE eagle SYSTEM "eagle.dtd">
-<eagle version="9.5.0">
+<eagle version="9.5.1">
 <drawing>
 <settings>
@@
 <wire x1="295.275" y1="40.005" x2="296.545" y2="41.275" width="0" layer="19" extent="16-16"/>
 </signal>
-<signal name="CONN_FPGA1:IN3_0">
+<signal name="CONN_FPGA1:IN2_0">
 <contactref element="CONN_FPGA1:J1" pad="H10"/>
 </signal>
-<signal name="CONN_FPGA1:IN3_1">
+<signal name="CONN_FPGA1:IN2_1">
 <contactref element="CONN_FPGA1:J1" pad="H11"/>
 </signal>
-<signal name="CONN_FPGA1:IN5_0">
+<signal name="CONN_FPGA1:IN4_0">
 <contactref element="CONN_FPGA1:J1" pad="H13"/>
 </signal>
-<signal name="CONN_FPGA1:IN5_1">
+<signal name="CONN_FPGA1:IN4_1">
 <contactref element="CONN_FPGA1:J1" pad="H14"/>
 </signal>
-<signal name="CONN_FPGA1:IN7_0">
+<signal name="CONN_FPGA1:IN6_0">
 <contactref element="CONN_FPGA1:J1" pad="H16"/>
 </signal>
-<signal name="CONN_FPGA1:IN7_1">
+<signal name="CONN_FPGA1:IN6_1">
 <contactref element="CONN_FPGA1:J1" pad="H17"/>
 </signal>
-<signal name="CONN_FPGA1:IN9_0">
+<signal name="CONN_FPGA1:IN8_0">
 <contactref element="CONN_FPGA1:J1" pad="H19"/>
 </signal>
-<signal name="CONN_FPGA1:IN9_1">
+<signal name="CONN_FPGA1:IN8_1">
 <contactref element="CONN_FPGA1:J1" pad="H20"/>
 </signal>
-<signal name="CONN_FPGA1:IN11_0">
+<signal name="CONN_FPGA1:IN10_0">
 <contactref element="CONN_FPGA1:J1" pad="H22"/>
 </signal>
-<signal name="CONN_FPGA1:IN11_1">
+<signal name="CONN_FPGA1:IN10_1">
 <contactref element="CONN_FPGA1:J1" pad="H23"/>
 </signal>
-<signal name="CONN_FPGA1:IN13_0">
-<contactref element="CONN_FPGA1:J1" pad="H25"/>
-</signal>
-<signal name="CONN_FPGA1:IN13_1">
-<contactref element="CONN_FPGA1:J1" pad="H26"/>
-</signal>
-<signal name="CONN_FPGA1:IN15_0">
-<contactref element="CONN_FPGA1:J1" pad="H28"/>
-</signal>
-<signal name="CONN_FPGA1:IN15_1">
-<contactref element="CONN_FPGA1:J1" pad="H29"/>
-</signal>
-<signal name="CONN_FPGA1:LA28_P">
-<contactref element="CONN_FPGA1:J1" pad="H31"/>
-</signal>
-<signal name="CONN_FPGA1:LA28_N">
-<contactref element="CONN_FPGA1:J1" pad="H32"/>
-</signal>
-<signal name="CONN_FPGA1:LA30_P">
-<contactref element="CONN_FPGA1:J1" pad="H34"/>
-</signal>
-<signal name="CONN_FPGA1:LA30_N">
-<contactref element="CONN_FPGA1:J1" pad="H35"/>
-</signal>
-<signal name="CONN_FPGA1:LA32_P">
-<contactref element="CONN_FPGA1:J1" pad="H37"/>
-</signal>
-<signal name="CONN_FPGA1:LA32_N">
-<contactref element="CONN_FPGA1:J1" pad="H38"/>
-</signal>
-<signal name="CONN_FPGA1:IN0_0">
-<contactref element="CONN_FPGA1:J1" pad="G6"/>
-</signal>
 <signal name="CONN_FPGA1:IN0_1">
-<contactref element="CONN_FPGA1:J1" pad="G7"/>
-</signal>
-<signal name="CONN_FPGA1:IN2_0">
-<contactref element="CONN_FPGA1:J1" pad="G9"/>
-</signal>
-<signal name="CONN_FPGA1:IN2_1">
-<contactref element="CONN_FPGA1:J1" pad="G10"/>
-</signal>
-<signal name="CONN_FPGA1:IN4_0">
-<contactref element="CONN_FPGA1:J1" pad="G12"/>
-</signal>
-<signal name="CONN_FPGA1:IN4_1">
-<contactref element="CONN_FPGA1:J1" pad="G13"/>
-</signal>
-<signal name="CONN_FPGA1:IN6_0">
-<contactref element="CONN_FPGA1:J1" pad="G15"/>
-</signal>
-<signal name="CONN_FPGA1:IN6_1">
-<contactref element="CONN_FPGA1:J1" pad="G16"/>
-</signal>
-<signal name="CONN_FPGA1:IN8_0">
-<contactref element="CONN_FPGA1:J1" pad="G18"/>
-</signal>
-<signal name="CONN_FPGA1:IN8_1">
-<contactref element="CONN_FPGA1:J1" pad="G19"/>
-</signal>
-<signal name="CONN_FPGA1:IN10_0">
-<contactref element="CONN_FPGA1:J1" pad="G21"/>
-</signal>
-<signal name="CONN_FPGA1:IN10_1">
-<contactref element="CONN_FPGA1:J1" pad="G22"/>
-</signal>
-<signal name="CONN_FPGA1:IN1_1">
 <contactref element="CONN_FPGA1:J1" pad="H8"/>
 </signal>
-<signal name="CONN_FPGA1:IN1_0">
+<signal name="CONN_FPGA1:IN0_0">
 <contactref element="CONN_FPGA1:J1" pad="H7"/>
 </signal>
 <signal name="CONN_FPGA1:IN12_0">
-<contactref element="CONN_FPGA1:J1" pad="G24"/>
+<contactref element="CONN_FPGA1:J1" pad="H25"/>
 </signal>
 <signal name="CONN_FPGA1:IN12_1">
-<contactref element="CONN_FPGA1:J1" pad="G25"/>
+<contactref element="CONN_FPGA1:J1" pad="H26"/>
 </signal>
 <signal name="CONN_FPGA1:IN14_0">
-<contactref element="CONN_FPGA1:J1" pad="G27"/>
+<contactref element="CONN_FPGA1:J1" pad="H28"/>
 </signal>
 <signal name="CONN_FPGA1:IN14_1">
-<contactref element="CONN_FPGA1:J1" pad="G28"/>
+<contactref element="CONN_FPGA1:J1" pad="H29"/>
 </signal>
 <signal name="POWER1:E1">
@@
 <contactref element="RECEIVER4:ADC2:ADC1" pad="24"/>
 </signal>
+<signal name="CONN_FPGA1:IN1_0">
+<contactref element="CONN_FPGA1:J1" pad="G9"/>
+</signal>
+<signal name="CONN_FPGA1:IN1_1">
+<contactref element="CONN_FPGA1:J1" pad="G10"/>
+</signal>
+<signal name="CONN_FPGA1:IN3_0">
+<contactref element="CONN_FPGA1:J1" pad="G12"/>
+</signal>
+<signal name="CONN_FPGA1:IN3_1">
+<contactref element="CONN_FPGA1:J1" pad="G13"/>
+</signal>
+<signal name="CONN_FPGA1:IN5_0">
+<contactref element="CONN_FPGA1:J1" pad="G15"/>
+</signal>
+<signal name="CONN_FPGA1:IN5_1">
+<contactref element="CONN_FPGA1:J1" pad="G16"/>
+</signal>
+<signal name="CONN_FPGA1:IN7_0">
+<contactref element="CONN_FPGA1:J1" pad="G18"/>
+</signal>
+<signal name="CONN_FPGA1:IN7_1">
+<contactref element="CONN_FPGA1:J1" pad="G19"/>
+</signal>
+<signal name="CONN_FPGA1:IN9_0">
+<contactref element="CONN_FPGA1:J1" pad="G21"/>
+</signal>
+<signal name="CONN_FPGA1:IN9_1">
+<contactref element="CONN_FPGA1:J1" pad="G22"/>
+</signal>
+<signal name="CONN_FPGA1:IN11_0">
+<contactref element="CONN_FPGA1:J1" pad="G24"/>
+</signal>
+<signal name="CONN_FPGA1:IN11_1">
+<contactref element="CONN_FPGA1:J1" pad="G25"/>
+</signal>
+<signal name="CONN_FPGA1:IN13_0">
+<contactref element="CONN_FPGA1:J1" pad="G27"/>
+</signal>
+<signal name="CONN_FPGA1:IN13_1">
+<contactref element="CONN_FPGA1:J1" pad="G28"/>
+</signal>
+<signal name="CONN_FPGA1:IN15_0">
+<contactref element="CONN_FPGA1:J1" pad="G30"/>
+</signal>
+<signal name="CONN_FPGA1:IN15_1">
+<contactref element="CONN_FPGA1:J1" pad="G31"/>
+</signal>
+<signal name="CONN_FPGA1:CW">
+<contactref element="CONN_FPGA1:J1" pad="H31"/>
+</signal>
+<signal name="CONN_FPGA1:SDO0_3">
+<contactref element="CONN_FPGA1:J1" pad="H34"/>
+</signal>
+<signal name="CONN_FPGA1:SDO0_2">
+<contactref element="CONN_FPGA1:J1" pad="H35"/>
+</signal>
+<signal name="CONN_FPGA1:SDO0_1">
+<contactref element="CONN_FPGA1:J1" pad="G33"/>
+</signal>
+<signal name="CONN_FPGA1:SDO0_0">
+<contactref element="CONN_FPGA1:J1" pad="G34"/>
+</signal>
+<signal name="CONN_FPGA1:CNV3">
+<contactref element="CONN_FPGA1:J1" pad="G37"/>
+</signal>
+<signal name="CONN_FPGA1:CNV2">
+<contactref element="CONN_FPGA1:J1" pad="G36"/>
+</signal>
+<signal name="CONN_FPGA1:CNV0">
+<contactref element="CONN_FPGA1:J1" pad="H37"/>
+</signal>
+<signal name="CONN_FPGA1:CNV1">
+<contactref element="CONN_FPGA1:J1" pad="H38"/>
+</signal>
+<signal name="CONN_FPGA1:SDO1_1">
+<contactref element="CONN_FPGA1:J1" pad="C10"/>
+</signal>
+<signal name="CONN_FPGA1:SDO1_0">
+<contactref element="CONN_FPGA1:J1" pad="C11"/>
+</signal>
+<signal name="CONN_FPGA1:SDO2_1">
+<contactref element="CONN_FPGA1:J1" pad="C14"/>
+</signal>
+<signal name="CONN_FPGA1:SDO2_0">
+<contactref element="CONN_FPGA1:J1" pad="C15"/>
+</signal>
+<signal name="CONN_FPGA1:SDO3_3">
+<contactref element="CONN_FPGA1:J1" pad="C18"/>
+</signal>
+<signal name="CONN_FPGA1:SDO3_2">
+<contactref element="CONN_FPGA1:J1" pad="C19"/>
+</signal>
+<signal name="CONN_FPGA1:SDO1_3">
+<contactref element="CONN_FPGA1:J1" pad="D11"/>
+</signal>
+<signal name="CONN_FPGA1:SDO1_2">
+<contactref element="CONN_FPGA1:J1" pad="D12"/>
+</signal>
+<signal name="CONN_FPGA1:SDO2_3">
+<contactref element="CONN_FPGA1:J1" pad="D14"/>
+</signal>
+<signal name="CONN_FPGA1:SDO2_2">
+<contactref element="CONN_FPGA1:J1" pad="D15"/>
+</signal>
+<signal name="CONN_FPGA1:SDO3_1">
+<contactref element="CONN_FPGA1:J1" pad="D17"/>
+</signal>
+<signal name="CONN_FPGA1:SDO3_0">
+<contactref element="CONN_FPGA1:J1" pad="D18"/>
+</signal>
+<signal name="CONN_FPGA1:SDI2">
+<contactref element="CONN_FPGA1:J1" pad="D23"/>
+</signal>
+<signal name="CONN_FPGA1:SDI3">
+<contactref element="CONN_FPGA1:J1" pad="D24"/>
+</signal>
+<signal name="CONN_FPGA1:BUSY2">
+<contactref element="CONN_FPGA1:J1" pad="C26"/>
+</signal>
+<signal name="CONN_FPGA1:BUSY3">
+<contactref element="CONN_FPGA1:J1" pad="C27"/>
+</signal>
+<signal name="CONN_FPGA1:ADC_CLK_1">
+<contactref element="CONN_FPGA1:J1" pad="G7"/>
+</signal>
+<signal name="CONN_FPGA1:ADC_CLK_0">
+<contactref element="CONN_FPGA1:J1" pad="G6"/>
+</signal>
+<signal name="CONN_FPGA1:ADC_CLK_2">
+<contactref element="CONN_FPGA1:J1" pad="H4"/>
+</signal>
+<signal name="CONN_FPGA1:SDI1">
+<contactref element="CONN_FPGA1:J1" pad="D21"/>
+</signal>
+<signal name="CONN_FPGA1:SDI0">
+<contactref element="CONN_FPGA1:J1" pad="D20"/>
+</signal>
+<signal name="CONN_FPGA1:BUSY0">
+<contactref element="CONN_FPGA1:J1" pad="D26"/>
+</signal>
+<signal name="CONN_FPGA1:BUSY1">
+<contactref element="CONN_FPGA1:J1" pad="D27"/>
+</signal>
+<signal name="CONN_FPGA1:CS0">
+<contactref element="CONN_FPGA1:J1" pad="D8"/>
+</signal>
+<signal name="CONN_FPGA1:CS1">
+<contactref element="CONN_FPGA1:J1" pad="D9"/>
+</signal>
+<signal name="CONN_FPGA1:CS2">
+<contactref element="CONN_FPGA1:J1" pad="C22"/>
+</signal>
+<signal name="CONN_FPGA1:CS3">
+<contactref element="CONN_FPGA1:J1" pad="C23"/>
+</signal>
+<signal name="CONN_FPGA1:ADC_CLK3">
+<contactref element="CONN_FPGA1:J1" pad="G2"/>
+</signal>
 </signals>

Commit message: schematic done except for power
Parts:
- removed CONN_FPGA1:C30: CBEC219-3479B001C1AF, wouter:BTB_CONN_68_F
- removed DRIVER1:C171, DRIVER1:C173, DRIVER1:C176, DRIVER1:C179, DRIVER1:C186, DRIVER1:C187, DRIVER1:C188, DRIVER1:C189, DRIVER2:C171, DRIVER2:C173, DRIVER2:C176, DRIVER2:C179, DRIVER2:C186, DRIVER2:C187, DRIVER2:C188, DRIVER2:C189: 220n 100V, rcl:C0805
- removed RECEIVER1:S12:C77, RECEIVER1:S12:C78, RECEIVER1:S5:C77, RECEIVER1:S5:C78, RECEIVER1:S6:C77, RECEIVER1:S6:C78, RECEIVER1:S7:C77, RECEIVER1:S7:C78, RECEIVER2:S12:C77, RECEIVER2:S12:C78, RECEIVER2:S5:C77, RECEIVER2:S5:C78, RECEIVER2:S6:C77, RECEIVER2:S6:C78, RECEIVER2:S7:C77, RECEIVER2:S7:C78, RECEIVER3:S12:C77, RECEIVER3:S12:C78, RECEIVER3:S5:C77, RECEIVER3:S5:C78, RECEIVER3:S6:C77, RECEIVER3:S6:C78, RECEIVER3:S7:C77, RECEIVER3:S7:C78, RECEIVER4:S12:C77, RECEIVER4:S12:C78, RECEIVER4:S5:C77, RECEIVER4:S5:C78, RECEIVER4:S6:C77, RECEIVER4:S6:C78, RECEIVER4:S7:C77, RECEIVER4:S7:C78: 100n, rcl:C050-025X075
- removed RECEIVER1:S12:D5, RECEIVER1:S12:D6, RECEIVER1:S5:D5, RECEIVER1:S5:D6, RECEIVER1:S6:D5, RECEIVER1:S6:D6, RECEIVER1:S7:D5, RECEIVER1:S7:D6, RECEIVER2:S12:D5, RECEIVER2:S12:D6, RECEIVER2:S5:D5, RECEIVER2:S5:D6, RECEIVER2:S6:D5, RECEIVER2:S6:D6, RECEIVER2:S7:D5, RECEIVER2:S7:D6, RECEIVER3:S12:D5, RECEIVER3:S12:D6, RECEIVER3:S5:D5, RECEIVER3:S5:D6, RECEIVER3:S6:D5, RECEIVER3:S6:D6, RECEIVER3:S7:D5, RECEIVER3:S7:D6, RECEIVER4:S12:D5, RECEIVER4:S12:D6, RECEIVER4:S5:D5, RECEIVER4:S5:D6, RECEIVER4:S6:D5, RECEIVER4:S6:D6, RECEIVER4:S7:D5, RECEIVER4:S7:D6: sbr3u20sa, dfls130l-7:POWERDI-123
- removed RECEIVER1:S12:R43, RECEIVER1:S12:R44, RECEIVER1:S5:R43, RECEIVER1:S5:R44, RECEIVER1:S6:R43, RECEIVER1:S6:R44, RECEIVER1:S7:R43, RECEIVER1:S7:R44, RECEIVER2:S12:R43, RECEIVER2:S12:R44, RECEIVER2:S5:R43, RECEIVER2:S5:R44, RECEIVER2:S6:R43, RECEIVER2:S6:R44, RECEIVER2:S7:R43, RECEIVER2:S7:R44, RECEIVER3:S12:R43, RECEIVER3:S12:R44, RECEIVER3:S5:R43, RECEIVER3:S5:R44, RECEIVER3:S6:R43, RECEIVER3:S6:R44, RECEIVER3:S7:R43, RECEIVER3:S7:R44, RECEIVER4:S12:R43, RECEIVER4:S12:R44, RECEIVER4:S5:R43, RECEIVER4:S5:R44, RECEIVER4:S6:R43, RECEIVER4:S6:R44, RECEIVER4:S7:R43, RECEIVER4:S7:R44: 1K, rcl:0207/7
- removed RECEIVER1:S12:SLIDESWITCH7, RECEIVER1:S5:SLIDESWITCH7, RECEIVER1:S6:SLIDESWITCH7, RECEIVER1:S7:SLIDESWITCH7, RECEIVER2:S12:SLIDESWITCH7, RECEIVER2:S5:SLIDESWITCH7, RECEIVER2:S6:SLIDESWITCH7, RECEIVER2:S7:SLIDESWITCH7, RECEIVER3:S12:SLIDESWITCH7, RECEIVER3:S5:SLIDESWITCH7, RECEIVER3:S6:SLIDESWITCH7, RECEIVER3:S7:SLIDESWITCH7, RECEIVER4:S12:SLIDESWITCH7, RECEIVER4:S5:SLIDESWITCH7, RECEIVER4:S6:SLIDESWITCH7, RECEIVER4:S7:SLIDESWITCH7: CL-SB-22A-01, wouter:CL-SB-22A-01
- removed RECEIVER1:S12:X12, RECEIVER1:S12:X2, RECEIVER1:S5:X12, RECEIVER1:S5:X2, RECEIVER1:S6:X12, RECEIVER1:S6:X2, RECEIVER1:S7:X12, RECEIVER1:S7:X2, RECEIVER2:S12:X12, RECEIVER2:S12:X2, RECEIVER2:S5:X12, RECEIVER2:S5:X2, RECEIVER2:S6:X12, RECEIVER2:S6:X2, RECEIVER2:S7:X12, RECEIVER2:S7:X2, RECEIVER3:S12:X12, RECEIVER3:S12:X2, RECEIVER3:S5:X12, RECEIVER3:S5:X2, RECEIVER3:S6:X12, RECEIVER3:S6:X2, RECEIVER3:S7:X12, RECEIVER3:S7:X2, RECEIVER4:S12:X12, RECEIVER4:S12:X2, RECEIVER4:S5:X12, RECEIVER4:S5:X2, RECEIVER4:S6:X12, RECEIVER4:S6:X2, RECEIVER4:S7:X12, RECEIVER4:S7:X2: (no value), con-phoenix-254:2POL254
- removed RECEIVER1:S1:C25, RECEIVER1:S1:C28, RECEIVER1:S2:C25, RECEIVER1:S2:C28, RECEIVER2:S1:C25, RECEIVER2:S1:C28, RECEIVER2:S2:C25, RECEIVER2:S2:C28, RECEIVER3:S1:C25, RECEIVER3:S1:C28, RECEIVER3:S2:C25, RECEIVER3:S2:C28, RECEIVER4:S1:C25, RECEIVER4:S1:C28, RECEIVER4:S2:C25, RECEIVER4:S2:C28: 18nF, rcl:C0603
- removed RECEIVER1:S1:GAIN12_1, RECEIVER1:S1:GAIN34_1, RECEIVER1:S2:GAIN12_1, RECEIVER1:S2:GAIN34_1, RECEIVER2:S1:GAIN12_1, RECEIVER2:S1:GAIN34_1, RECEIVER2:S2:GAIN12_1, RECEIVER2:S2:GAIN34_1, RECEIVER3:S1:GAIN12_1, RECEIVER3:S1:GAIN34_1, RECEIVER3:S2:GAIN12_1, RECEIVER3:S2:GAIN34_1, RECEIVER4:S1:GAIN12_1, RECEIVER4:S1:GAIN34_1, RECEIVER4:S2:GAIN12_1, RECEIVER4:S2:GAIN34_1: 3361S-1-104GLF, 3361S-1-104GLF:3361S
- removed RECEIVER1:S1:JP1, RECEIVER1:S1:JP2, RECEIVER1:S2:JP1, RECEIVER1:S2:JP2, RECEIVER2:S1:JP1, RECEIVER2:S1:JP2, RECEIVER2:S2:JP1, RECEIVER2:S2:JP2, RECEIVER3:S1:JP1, RECEIVER3:S1:JP2, RECEIVER3:S2:JP1, RECEIVER3:S2:JP2, RECEIVER4:S1:JP1, RECEIVER4:S1:JP2, RECEIVER4:S2:JP1, RECEIVER4:S2:JP2: (no value), jumper:JP1
- removed RECEIVER1:S1:SLIDESWITCH1, RECEIVER1:S1:SLIDESWITCH2, RECEIVER1:S2:SLIDESWITCH1, RECEIVER1:S2:SLIDESWITCH2, RECEIVER2:S1:SLIDESWITCH1, RECEIVER2:S1:SLIDESWITCH2, RECEIVER2:S2:SLIDESWITCH1, RECEIVER2:S2:SLIDESWITCH2, RECEIVER3:S1:SLIDESWITCH1, RECEIVER3:S1:SLIDESWITCH2, RECEIVER3:S2:SLIDESWITCH1, RECEIVER3:S2:SLIDESWITCH2, RECEIVER4:S1:SLIDESWITCH1, RECEIVER4:S1:SLIDESWITCH2, RECEIVER4:S2:SLIDESWITCH1, RECEIVER4:S2:SLIDESWITCH2: CL-SB-12A-01, wouter:CL-SB-12A-01
- added CONN_RESONATORS1:C30: CBEC219-3479B001C1AF, wouter:BTB_CONN_68_F
- added RECEIVER1:ADC2:R1, RECEIVER1:ADC2:R2, RECEIVER1:ADC2:R3, RECEIVER1:ADC2:R4, RECEIVER1:ADC2:R5, RECEIVER1:ADC2:R6, RECEIVER1:ADC2:R7, RECEIVER2:ADC2:R1, RECEIVER2:ADC2:R2, RECEIVER2:ADC2:R3, RECEIVER2:ADC2:R4, RECEIVER2:ADC2:R5, RECEIVER2:ADC2:R6, RECEIVER2:ADC2:R7, RECEIVER3:ADC2:R1, RECEIVER3:ADC2:R2, RECEIVER3:ADC2:R3, RECEIVER3:ADC2:R4, RECEIVER3:ADC2:R5, RECEIVER3:ADC2:R6, RECEIVER3:ADC2:R7, RECEIVER4:ADC2:R1, RECEIVER4:ADC2:R2, RECEIVER4:ADC2:R3, RECEIVER4:ADC2:R4, RECEIVER4:ADC2:R5, RECEIVER4:ADC2:R6, RECEIVER4:ADC2:R7: 33R, rcl:R0402
- added RECEIVER1:S12:C1, RECEIVER1:S12:C2, RECEIVER1:S5:C1, RECEIVER1:S5:C2, RECEIVER1:S6:C1, RECEIVER1:S6:C2, RECEIVER1:S7:C1, RECEIVER1:S7:C2, RECEIVER2:S12:C1, RECEIVER2:S12:C2, RECEIVER2:S5:C1, RECEIVER2:S5:C2, RECEIVER2:S6:C1, RECEIVER2:S6:C2, RECEIVER2:S7:C1, RECEIVER2:S7:C2, RECEIVER3:S12:C1, RECEIVER3:S12:C2, RECEIVER3:S5:C1, RECEIVER3:S5:C2, RECEIVER3:S6:C1, RECEIVER3:S6:C2, RECEIVER3:S7:C1, RECEIVER3:S7:C2, RECEIVER4:S12:C1, RECEIVER4:S12:C2, RECEIVER4:S5:C1, RECEIVER4:S5:C2, RECEIVER4:S6:C1, RECEIVER4:S6:C2, RECEIVER4:S7:C1, RECEIVER4:S7:C2: 100n, rcl:C0603
- added RECEIVER1:S12:C3, RECEIVER1:S12:C4, RECEIVER1:S5:C3, RECEIVER1:S5:C4, RECEIVER1:S6:C3, RECEIVER1:S6:C4, RECEIVER1:S7:C3, RECEIVER1:S7:C4, RECEIVER2:S12:C3, RECEIVER2:S12:C4, RECEIVER2:S5:C3, RECEIVER2:S5:C4, RECEIVER2:S6:C3, RECEIVER2:S6:C4, RECEIVER2:S7:C3, RECEIVER2:S7:C4, RECEIVER3:S12:C3, RECEIVER3:S12:C4, RECEIVER3:S5:C3, RECEIVER3:S5:C4, RECEIVER3:S6:C3, RECEIVER3:S6:C4, RECEIVER3:S7:C3, RECEIVER3:S7:C4, RECEIVER4:S12:C3, RECEIVER4:S12:C4, RECEIVER4:S5:C3, RECEIVER4:S5:C4, RECEIVER4:S6:C3, RECEIVER4:S6:C4, RECEIVER4:S7:C3, RECEIVER4:S7:C4: 100n C0G, rcl:C1206
- added RECEIVER1:S12:C5, RECEIVER1:S12:C6, RECEIVER1:S5:C5, RECEIVER1:S5:C6, RECEIVER1:S6:C5, RECEIVER1:S6:C6, RECEIVER1:S7:C5, RECEIVER1:S7:C6, RECEIVER2:S12:C5, RECEIVER2:S12:C6, RECEIVER2:S5:C5, RECEIVER2:S5:C6, RECEIVER2:S6:C5, RECEIVER2:S6:C6, RECEIVER2:S7:C5, RECEIVER2:S7:C6, RECEIVER3:S12:C5, RECEIVER3:S12:C6, RECEIVER3:S5:C5, RECEIVER3:S5:C6, RECEIVER3:S6:C5, RECEIVER3:S6:C6, RECEIVER3:S7:C5, RECEIVER3:S7:C6, RECEIVER4:S12:C5, RECEIVER4:S12:C6, RECEIVER4:S5:C5, RECEIVER4:S5:C6, RECEIVER4:S6:C5, RECEIVER4:S6:C6, RECEIVER4:S7:C5, RECEIVER4:S7:C6: 3.3u, rcl:C0402
- added RECEIVER1:S12:D1, RECEIVER1:S12:D2, RECEIVER1:S5:D1, RECEIVER1:S5:D2, RECEIVER1:S6:D1, RECEIVER1:S6:D2, RECEIVER1:S7:D1, RECEIVER1:S7:D2, RECEIVER2:S12:D1, RECEIVER2:S12:D2, RECEIVER2:S5:D1, RECEIVER2:S5:D2, RECEIVER2:S6:D1, RECEIVER2:S6:D2, RECEIVER2:S7:D1, RECEIVER2:S7:D2, RECEIVER3:S12:D1, RECEIVER3:S12:D2, RECEIVER3:S5:D1, RECEIVER3:S5:D2, RECEIVER3:S6:D1, RECEIVER3:S6:D2, RECEIVER3:S7:D1, RECEIVER3:S7:D2, RECEIVER4:S12:D1, RECEIVER4:S12:D2, RECEIVER4:S5:D1, RECEIVER4:S5:D2, RECEIVER4:S6:D1, RECEIVER4:S6:D2, RECEIVER4:S7:D1, RECEIVER4:S7:D2: MBR0520L, wouter:SOD3816X128N
- added RECEIVER1:S12:IC1, RECEIVER1:S5:IC1, RECEIVER1:S6:IC1, RECEIVER1:S7:IC1, RECEIVER2:S12:IC1, RECEIVER2:S5:IC1, RECEIVER2:S6:IC1, RECEIVER2:S7:IC1, RECEIVER3:S12:IC1, RECEIVER3:S5:IC1, RECEIVER3:S6:IC1, RECEIVER3:S7:IC1, RECEIVER4:S12:IC1, RECEIVER4:S5:IC1, RECEIVER4:S6:IC1, RECEIVER4:S7:IC1: LT6238HGN#PBF, wouter:SOP64P601X175-16N
- added RECEIVER1:S12:R1, RECEIVER1:S12:R2, RECEIVER1:S5:R1, RECEIVER1:S5:R2, RECEIVER1:S6:R1, RECEIVER1:S6:R2, RECEIVER1:S7:R1, RECEIVER1:S7:R2, RECEIVER2:S12:R1, RECEIVER2:S12:R2, RECEIVER2:S5:R1, RECEIVER2:S5:R2, RECEIVER2:S6:R1, RECEIVER2:S6:R2, RECEIVER2:S7:R1, RECEIVER2:S7:R2, RECEIVER3:S12:R1, RECEIVER3:S12:R2, RECEIVER3:S5:R1, RECEIVER3:S5:R2, RECEIVER3:S6:R1, RECEIVER3:S6:R2, RECEIVER3:S7:R1, RECEIVER3:S7:R2, RECEIVER4:S12:R1, RECEIVER4:S12:R2, RECEIVER4:S5:R1, RECEIVER4:S5:R2, RECEIVER4:S6:R1, RECEIVER4:S6:R2, RECEIVER4:S7:R1, RECEIVER4:S7:R2: 300R, rcl:M0805
- added RECEIVER1:S12:R3, RECEIVER1:S12:R4, RECEIVER1:S5:R3, RECEIVER1:S5:R4, RECEIVER1:S6:R3, RECEIVER1:S6:R4, RECEIVER1:S7:R3, RECEIVER1:S7:R4, RECEIVER2:S12:R3, RECEIVER2:S12:R4, RECEIVER2:S5:R3, RECEIVER2:S5:R4, RECEIVER2:S6:R3, RECEIVER2:S6:R4, RECEIVER2:S7:R3, RECEIVER2:S7:R4, RECEIVER3:S12:R3, RECEIVER3:S12:R4, RECEIVER3:S5:R3, RECEIVER3:S5:R4, RECEIVER3:S6:R3, RECEIVER3:S6:R4, RECEIVER3:S7:R3, RECEIVER3:S7:R4, RECEIVER4:S12:R3, RECEIVER4:S12:R4, RECEIVER4:S5:R3, RECEIVER4:S5:R4, RECEIVER4:S6:R3, RECEIVER4:S6:R4, RECEIVER4:S7:R3, RECEIVER4:S7:R4: 82R, rcl:M0805
- added RECEIVER1:S1:C11, RECEIVER1:S1:C12, RECEIVER1:S2:C11, RECEIVER1:S2:C12, RECEIVER2:S1:C11, RECEIVER2:S1:C12, RECEIVER2:S2:C11, RECEIVER2:S2:C12, RECEIVER3:S1:C11, RECEIVER3:S1:C12, RECEIVER3:S2:C11, RECEIVER3:S2:C12, RECEIVER4:S1:C11, RECEIVER4:S1:C12, RECEIVER4:S2:C11, RECEIVER4:S2:C12: 18nF, Wurth_Elektronik_Passive_Capacitors_rev18b:WCAP-CSGP_0402
- added RECEIVER1:S1:R10, RECEIVER1:S2:R10, RECEIVER2:S1:R10, RECEIVER2:S2:R10, RECEIVER3:S1:R10, RECEIVER3:S2:R10, RECEIVER4:S1:R10, RECEIVER4:S2:R10: DNP, resistor:R0402
- added RECEIVER1:S1:R11, RECEIVER1:S1:R2, RECEIVER1:S2:R11, RECEIVER1:S2:R2, RECEIVER2:S1:R11, RECEIVER2:S1:R2, RECEIVER2:S2:R11, RECEIVER2:S2:R2, RECEIVER3:S1:R11, RECEIVER3:S1:R2, RECEIVER3:S2:R11, RECEIVER3:S2:R2, RECEIVER4:S1:R11, RECEIVER4:S1:R2, RECEIVER4:S2:R11, RECEIVER4:S2:R2: 0R, resistor:R0402
- added RECEIVER1:S1:R12, RECEIVER1:S1:R15, RECEIVER1:S2:R12, RECEIVER1:S2:R15, RECEIVER2:S1:R12, RECEIVER2:S1:R15, RECEIVER2:S2:R12, RECEIVER2:S2:R15, RECEIVER3:S1:R12, RECEIVER3:S1:R15, RECEIVER3:S2:R12, RECEIVER3:S2:R15, RECEIVER4:S1:R12, RECEIVER4:S1:R15, RECEIVER4:S2:R12, RECEIVER4:S2:R15: 274R, resistor:R0402
- added RECEIVER1:S1:R13, RECEIVER1:S2:R13, RECEIVER2:S1:R13, RECEIVER2:S2:R13, RECEIVER3:S1:R13, RECEIVER3:S2:R13, RECEIVER4:S1:R13, RECEIVER4:S2:R13: 1K, resistor:R0402
- added RECEIVER1:S1:VR1, RECEIVER1:S1:VR2, RECEIVER1:S2:VR1, RECEIVER1:S2:VR2, RECEIVER2:S1:VR1, RECEIVER2:S1:VR2, RECEIVER2:S2:VR1, RECEIVER2:S2:VR2, RECEIVER3:S1:VR1, RECEIVER3:S1:VR2, RECEIVER3:S2:VR1, RECEIVER3:S2:VR2, RECEIVER4:S1:VR1, RECEIVER4:S1:VR2, RECEIVER4:S2:VR1, RECEIVER4:S2:VR2: 10k, SparkFun-Resistors:TRIMPOT-SMD-TC33X
- RECEIVER1:ADC2:C140, RECEIVER2:ADC2:C140, RECEIVER3:ADC2:C140, RECEIVER4:ADC2:C140: value 47uf -> 47uf 10V
- RECEIVER1:S1:C19, RECEIVER1:S1:C20, RECEIVER1:S2:C19, RECEIVER1:S2:C20, RECEIVER2:S1:C19, RECEIVER2:S1:C20, RECEIVER2:S2:C19, RECEIVER2:S2:C20, RECEIVER3:S1:C19, RECEIVER3:S1:C20, RECEIVER3:S2:C19, RECEIVER3:S2:C20, RECEIVER4:S1:C19, RECEIVER4:S1:C20, RECEIVER4:S2:C19, RECEIVER4:S2:C20: value 1nF -> 10nF; device rcl:C0402 -> Wurth_Elektronik_Passive_Capacitors_rev18b:WCAP-CSGP_0402
- RECEIVER1:S1:R1, RECEIVER1:S1:R3, RECEIVER1:S2:R1, RECEIVER1:S2:R3, RECEIVER2:S1:R1, RECEIVER2:S1:R3, RECEIVER2:S2:R1, RECEIVER2:S2:R3, RECEIVER3:S1:R1, RECEIVER3:S1:R3, RECEIVER3:S2:R1, RECEIVER3:S2:R3, RECEIVER4:S1:R1, RECEIVER4:S1:R3, RECEIVER4:S2:R1, RECEIVER4:S2:R3: value 400k -> 39K; device resistor:R0603 -> resistor:R0402
- RECEIVER1:S1:R4, RECEIVER1:S1:R5, RECEIVER1:S2:R4, RECEIVER1:S2:R5, RECEIVER2:S1:R4, RECEIVER2:S1:R5, RECEIVER2:S2:R4, RECEIVER2:S2:R5, RECEIVER3:S1:R4, RECEIVER3:S1:R5, RECEIVER3:S2:R4, RECEIVER3:S2:R5, RECEIVER4:S1:R4, RECEIVER4:S1:R5, RECEIVER4:S2:R4, RECEIVER4:S2:R5: value 4.02k -> 4K02; device resistor:R0805 -> resistor:R0402
- RECEIVER1:S1:R6, RECEIVER1:S2:R6, RECEIVER2:S1:R6, RECEIVER2:S2:R6, RECEIVER3:S1:R6, RECEIVER3:S2:R6, RECEIVER4:S1:R6, RECEIVER4:S2:R6: value 274 -> DNP; device resistor:R0603 -> resistor:R0402
- RECEIVER1:S1:R7, RECEIVER1:S2:R7, RECEIVER2:S1:R7, RECEIVER2:S2:R7, RECEIVER3:S1:R7, RECEIVER3:S2:R7, RECEIVER4:S1:R7, RECEIVER4:S2:R7: value 274 -> 0R; device resistor:R0603 -> resistor:R0402
- RECEIVER1:S1:R8, RECEIVER1:S2:R8, RECEIVER2:S1:R8, RECEIVER2:S2:R8, RECEIVER3:S1:R8, RECEIVER3:S2:R8, RECEIVER4:S1:R8, RECEIVER4:S2:R8: device resistor:R0603 -> resistor:R0402
- RECEIVER1:S1:R9, RECEIVER1:S2:R9, RECEIVER2:S1:R9, RECEIVER2:S2:R9, RECEIVER3:S1:R9, RECEIVER3:S2:R9, RECEIVER4:S1:R9, RECEIVER4:S2:R9: value 0R -> 1K; device resistor:R0603 -> resistor:R0402
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Connections:
- net RECEIVER1:!CS renamed RECEIVER1:ADC2:/CS
- net RECEIVER1:ADC2:3V3 renamed RECEIVER1:ADC2:OVDD
- net RECEIVER1:ADC2:5V renamed RECEIVER1:ADC2:+5V
- net RECEIVER1:ADC2:ADIN1_N renamed RECEIVER1:ADC2:ADIN0_N
- net RECEIVER2:!CS renamed RECEIVER2:ADC2:/CS
- net RECEIVER2:ADC2:3V3 renamed RECEIVER2:ADC2:OVDD
- net RECEIVER2:ADC2:5V renamed RECEIVER2:ADC2:+5V
- net RECEIVER2:ADC2:ADIN1_N renamed RECEIVER2:ADC2:ADIN0_N
- net RECEIVER3:!CS renamed RECEIVER3:ADC2:/CS
- net RECEIVER3:ADC2:3V3 renamed RECEIVER3:ADC2:OVDD
- net RECEIVER3:ADC2:5V renamed RECEIVER3:ADC2:+5V
- net RECEIVER3:ADC2:ADIN1_N renamed RECEIVER3:ADC2:ADIN0_N
- net RECEIVER4:!CS renamed RECEIVER4:ADC2:/CS
- net RECEIVER4:ADC2:3V3 renamed RECEIVER4:ADC2:OVDD
- net RECEIVER4:ADC2:5V renamed RECEIVER4:ADC2:+5V
- net RECEIVER4:ADC2:ADIN1_N renamed RECEIVER4:ADC2:ADIN0_N
- removed net CONN_FPGA1:ADC_CLK3: CONN_FPGA1:J1.G2
- removed net CONN_FPGA1:ADC_CLK_0: CONN_FPGA1:J1.G6
- removed net CONN_FPGA1:ADC_CLK_1: CONN_FPGA1:J1.G7
- removed net CONN_FPGA1:ADC_CLK_2: CONN_FPGA1:J1.H4
- removed net CONN_FPGA1:BUSY0: CONN_FPGA1:J1.D26
- removed net CONN_FPGA1:BUSY1: CONN_FPGA1:J1.D27
- removed net CONN_FPGA1:BUSY2: CONN_FPGA1:J1.C26
- removed net CONN_FPGA1:BUSY3: CONN_FPGA1:J1.C27
- removed net CONN_FPGA1:CNV0: CONN_FPGA1:J1.H37
- removed net CONN_FPGA1:CNV1: CONN_FPGA1:J1.H38
- removed net CONN_FPGA1:CNV2: CONN_FPGA1:J1.G36
- removed net CONN_FPGA1:CNV3: CONN_FPGA1:J1.G37
- removed net CONN_FPGA1:CS0: CONN_FPGA1:J1.D8
- removed net CONN_FPGA1:CS1: CONN_FPGA1:J1.D9
- removed net CONN_FPGA1:CS2: CONN_FPGA1:J1.C22
- removed net CONN_FPGA1:CS3: CONN_FPGA1:J1.C23
- removed net CONN_FPGA1:CW: CONN_FPGA1:J1.H31
- removed net CONN_FPGA1:IN0_0: CONN_FPGA1:J1.H7
- removed net CONN_FPGA1:IN0_1: CONN_FPGA1:J1.H8
- removed net CONN_FPGA1:IN10_0: CONN_FPGA1:J1.H22
- removed net CONN_FPGA1:IN10_1: CONN_FPGA1:J1.H23
- removed net CONN_FPGA1:IN11_0: CONN_FPGA1:J1.G24
- removed net CONN_FPGA1:IN11_1: CONN_FPGA1:J1.G25
- removed net CONN_FPGA1:IN12_0: CONN_FPGA1:J1.H25
- removed net CONN_FPGA1:IN12_1: CONN_FPGA1:J1.H26
- removed net CONN_FPGA1:IN13_0: CONN_FPGA1:J1.G27
- removed net CONN_FPGA1:IN13_1: CONN_FPGA1:J1.G28
- removed net CONN_FPGA1:IN14_0: CONN_FPGA1:J1.H28
- removed net CONN_FPGA1:IN14_1: CONN_FPGA1:J1.H29
- removed net CONN_FPGA1:IN15_0: CONN_FPGA1:J1.G30
- removed net CONN_FPGA1:IN15_1: CONN_FPGA1:J1.G31
- removed net CONN_FPGA1:IN1_0: CONN_FPGA1:J1.G9
- removed net CONN_FPGA1:IN1_1: CONN_FPGA1:J1.G10
- removed net CONN_FPGA1:IN2_0: CONN_FPGA1:J1.H10
- removed net CONN_FPGA1:IN2_1: CONN_FPGA1:J1.H11
- removed net CONN_FPGA1:IN3_0: CONN_FPGA1:J1.G12
- removed net CONN_FPGA1:IN3_1: CONN_FPGA1:J1.G13
- removed net CONN_FPGA1:IN4_0: CONN_FPGA1:J1.H13
- removed net CONN_FPGA1:IN4_1: CONN_FPGA1:J1.H14
- removed net CONN_FPGA1:IN5_0: CONN_FPGA1:J1.G15
- removed net CONN_FPGA1:IN5_1: CONN_FPGA1:J1.G16
- removed net CONN_FPGA1:IN6_0: CONN_FPGA1:J1.H16
- removed net CONN_FPGA1:IN6_1: CONN_FPGA1:J1.H17
- removed net CONN_FPGA1:IN7_0: CONN_FPGA1:J1.G18
- removed net CONN_FPGA1:IN7_1: CONN_FPGA1:J1.G19
- removed net CONN_FPGA1:IN8_0: CONN_FPGA1:J1.H19
- removed net CONN_FPGA1:IN8_1: CONN_FPGA1:J1.H20
- removed net CONN_FPGA1:IN9_0: CONN_FPGA1:J1.G21
- removed net CONN_FPGA1:IN9_1: CONN_FPGA1:J1.G22
- removed net CONN_FPGA1:OUT_0: CONN_FPGA1:C30.2
- removed net CONN_FPGA1:OUT_1: CONN_FPGA1:C30.3
- removed net CONN_FPGA1:OUT_10: CONN_FPGA1:C30.12
- removed net CONN_FPGA1:OUT_11: CONN_FPGA1:C30.13
- removed net CONN_FPGA1:OUT_12: CONN_FPGA1:C30.14
- removed net CONN_FPGA1:OUT_13: CONN_FPGA1:C30.15
- removed net CONN_FPGA1:OUT_14: CONN_FPGA1:C30.16
- removed net CONN_FPGA1:OUT_15: CONN_FPGA1:C30.17
- removed net CONN_FPGA1:OUT_16: CONN_FPGA1:C30.18
- removed net CONN_FPGA1:OUT_17: CONN_FPGA1:C30.19
- removed net CONN_FPGA1:OUT_18: CONN_FPGA1:C30.20
- removed net CONN_FPGA1:OUT_19: CONN_FPGA1:C30.21
- removed net CONN_FPGA1:OUT_2: CONN_FPGA1:C30.4
- removed net CONN_FPGA1:OUT_20: CONN_FPGA1:C30.22
- removed net CONN_FPGA1:OUT_21: CONN_FPGA1:C30.23
- removed net CONN_FPGA1:OUT_22: CONN_FPGA1:C30.24
- removed net CONN_FPGA1:OUT_23: CONN_FPGA1:C30.25
- removed net CONN_FPGA1:OUT_24: CONN_FPGA1:C30.26
- removed net CONN_FPGA1:OUT_25: CONN_FPGA1:C30.27
- removed net CONN_FPGA1:OUT_26: CONN_FPGA1:C30.28
- removed net CONN_FPGA1:OUT_27: CONN_FPGA1:C30.29
- removed net CONN_FPGA1:OUT_28: CONN_FPGA1:C30.30
- removed net CONN_FPGA1:OUT_29: CONN_FPGA1:C30.31
- removed net CONN_FPGA1:OUT_3: CONN_FPGA1:C30.5
- removed net CONN_FPGA1:OUT_30: CONN_FPGA1:C30.32
- removed net CONN_FPGA1:OUT_31: CONN_FPGA1:C30.33
- removed net CONN_FPGA1:OUT_32: CONN_FPGA1:C30.36
- removed net CONN_FPGA1:OUT_33: CONN_FPGA1:C30.37
- removed net CONN_FPGA1:OUT_34: CONN_FPGA1:C30.38
- removed net CONN_FPGA1:OUT_35: CONN_FPGA1:C30.39
- removed net CONN_FPGA1:OUT_36: CONN_FPGA1:C30.40
- removed net CONN_FPGA1:OUT_37: CONN_FPGA1:C30.41
- removed net CONN_FPGA1:OUT_38: CONN_FPGA1:C30.42
- removed net CONN_FPGA1:OUT_39: CONN_FPGA1:C30.43
- removed net CONN_FPGA1:OUT_4: CONN_FPGA1:C30.6
- removed net CONN_FPGA1:OUT_40: CONN_FPGA1:C30.44
- removed net CONN_FPGA1:OUT_41: CONN_FPGA1:C30.45
- removed net CONN_FPGA1:OUT_42: CONN_FPGA1:C30.46
- removed net CONN_FPGA1:OUT_43: CONN_FPGA1:C30.47
- removed net CONN_FPGA1:OUT_44: CONN_FPGA1:C30.48
- removed net CONN_FPGA1:OUT_45: CONN_FPGA1:C30.49
- removed net CONN_FPGA1:OUT_46: CONN_FPGA1:C30.50
- removed net CONN_FPGA1:OUT_47: CONN_FPGA1:C30.51
- removed net CONN_FPGA1:OUT_48: CONN_FPGA1:C30.52
- removed net CONN_FPGA1:OUT_49: CONN_FPGA1:C30.53
- removed net CONN_FPGA1:OUT_5: CONN_FPGA1:C30.7
- removed net CONN_FPGA1:OUT_50: CONN_FPGA1:C30.54
- removed net CONN_FPGA1:OUT_51: CONN_FPGA1:C30.55
- removed net CONN_FPGA1:OUT_52: CONN_FPGA1:C30.56
- removed net CONN_FPGA1:OUT_53: CONN_FPGA1:C30.57
- removed net CONN_FPGA1:OUT_54: CONN_FPGA1:C30.58
- removed net CONN_FPGA1:OUT_55: CONN_FPGA1:C30.59
- removed net CONN_FPGA1:OUT_56: CONN_FPGA1:C30.60
- removed net CONN_FPGA1:OUT_57: CONN_FPGA1:C30.61
- removed net CONN_FPGA1:OUT_58: CONN_FPGA1:C30.62
- removed net CONN_FPGA1:OUT_59: CONN_FPGA1:C30.63
- removed net CONN_FPGA1:OUT_6: CONN_FPGA1:C30.8
- removed net CONN_FPGA1:OUT_60: CONN_FPGA1:C30.64
- removed net CONN_FPGA1:OUT_61: CONN_FPGA1:C30.65
- removed net CONN_FPGA1:OUT_62: CONN_FPGA1:C30.66
- removed net CONN_FPGA1:OUT_63: CONN_FPGA1:C30.67
- removed net CONN_FPGA1:OUT_7: CONN_FPGA1:C30.9
- removed net CONN_FPGA1:OUT_8: CONN_FPGA1:C30.10
- removed net CONN_FPGA1:OUT_9: CONN_FPGA1:C30.11
- removed net CONN_FPGA1:SDI0: CONN_FPGA1:J1.D20
- removed net CONN_FPGA1:SDI1: CONN_FPGA1:J1.D21
- removed net CONN_FPGA1:SDI2: CONN_FPGA1:J1.D23
- removed net CONN_FPGA1:SDI3: CONN_FPGA1:J1.D24
- removed net CONN_FPGA1:SDO0_0: CONN_FPGA1:J1.G34
- removed net CONN_FPGA1:SDO0_1: CONN_FPGA1:J1.G33
- removed net CONN_FPGA1:SDO0_2: CONN_FPGA1:J1.H35
- removed net CONN_FPGA1:SDO0_3: CONN_FPGA1:J1.H34
- removed net CONN_FPGA1:SDO1_0: CONN_FPGA1:J1.C11
- removed net CONN_FPGA1:SDO1_1: CONN_FPGA1:J1.C10
- removed net CONN_FPGA1:SDO1_2: CONN_FPGA1:J1.D12
- removed net CONN_FPGA1:SDO1_3: CONN_FPGA1:J1.D11
- removed net CONN_FPGA1:SDO2_0: CONN_FPGA1:J1.C15
- removed net CONN_FPGA1:SDO2_1: CONN_FPGA1:J1.C14
- removed net CONN_FPGA1:SDO2_2: CONN_FPGA1:J1.D15
- removed net CONN_FPGA1:SDO2_3: CONN_FPGA1:J1.D14
- removed net CONN_FPGA1:SDO3_0: CONN_FPGA1:J1.D18
- removed net CONN_FPGA1:SDO3_1: CONN_FPGA1:J1.D17
- removed net CONN_FPGA1:SDO3_2: CONN_FPGA1:J1.C19
- removed net CONN_FPGA1:SDO3_3: CONN_FPGA1:J1.C18
- removed net DRIVER1:CW: DRIVER1:STHV_0.CW
- removed net DRIVER1:DVDD: DRIVER1:C182.1, DRIVER1:R2.2, DRIVER1:STHV_0.DVDD
- removed net DRIVER1:IN0_0: DRIVER1:STHV_0.IN1_0
- removed net DRIVER1:IN0_1: DRIVER1:STHV_0.IN1_1
- removed net DRIVER1:IN1_0: DRIVER1:STHV_0.IN2_0
- removed net DRIVER1:IN1_1: DRIVER1:STHV_0.IN2_1
- removed net DRIVER1:IN2_0: DRIVER1:STHV_0.IN3_0
- removed net DRIVER1:IN2_1: DRIVER1:STHV_0.IN3_1
- removed net DRIVER1:IN3_0: DRIVER1:STHV_0.IN4_0
- removed net DRIVER1:IN3_1: DRIVER1:STHV_0.IN4_1
- removed net DRIVER1:IN4_0: DRIVER1:STHV_0.IN5_0
- removed net DRIVER1:IN4_1: DRIVER1:STHV_0.IN5_1
- removed net DRIVER1:IN5_0: DRIVER1:STHV_0.IN6_0
- removed net DRIVER1:IN5_1: DRIVER1:STHV_0.IN6_1
- removed net DRIVER1:IN6_0: DRIVER1:STHV_0.IN7_0
- removed net DRIVER1:IN6_1: DRIVER1:STHV_0.IN7_1
- removed net DRIVER1:IN7_0: DRIVER1:STHV_0.IN8_0
- removed net DRIVER1:IN7_1: DRIVER1:STHV_0.IN8_1
- removed net DRIVER1:INX_1_0: DRIVER1:IN0_1.1
- removed net DRIVER1:LVOUT_0: DRIVER1:LVOUT0.1, DRIVER1:STHV_0.LVOUT_1
- removed net DRIVER1:LVOUT_1: DRIVER1:STHV_0.LVOUT_2
- removed net DRIVER1:LVOUT_2: DRIVER1:STHV_0.LVOUT_3
- removed net DRIVER1:LVOUT_3: DRIVER1:STHV_0.LVOUT_4
- removed net DRIVER1:LVOUT_4: DRIVER1:STHV_0.LVOUT_5
- removed net DRIVER1:LVOUT_5: DRIVER1:STHV_0.LVOUT_6
- removed net DRIVER1:LVOUT_6: DRIVER1:STHV_0.LVOUT_7
- removed net DRIVER1:LVOUT_7: DRIVER1:STHV_0.LVOUT_8
- removed net DRIVER1:OUT_0: DRIVER1:D0_0.A, DRIVER1:D0_1.C, DRIVER1:STHV_0.XDCR_1, DRIVER1:T_OUT_0.1
- removed net DRIVER1:OUT_1: DRIVER1:D1_0.A, DRIVER1:D1_1.C, DRIVER1:STHV_0.XDCR_2, DRIVER1:T_OUT_1.1
- removed net DRIVER1:OUT_2: DRIVER1:D2_0.A, DRIVER1:D2_1.C, DRIVER1:STHV_0.XDCR_3, DRIVER1:T_OUT_2.1
- removed net DRIVER1:OUT_3: DRIVER1:D3_0.A, DRIVER1:D3_1.C, DRIVER1:STHV_0.XDCR_4, DRIVER1:T_OUT_3.1
- removed net DRIVER1:OUT_4: DRIVER1:D4_0.A, DRIVER1:D4_1.C, DRIVER1:STHV_0.XDCR_5, DRIVER1:T_OUT_4.1
- removed net DRIVER1:OUT_5: DRIVER1:D5_0.A, DRIVER1:D5_1.C, DRIVER1:STHV_0.XDCR_6, DRIVER1:T_OUT_5.1
- removed net DRIVER1:OUT_6: DRIVER1:D6_0.A, DRIVER1:D6_1.C, DRIVER1:STHV_0.XDCR_7, DRIVER1:T_OUT_6.1
- removed net DRIVER1:OUT_7: DRIVER1:D7_0.A, DRIVER1:D7_1.C, DRIVER1:STHV_0.XDCR_8, DRIVER1:T_OUT_7.1
- removed net DRIVER1:PWM_INT0: DRIVER1:IN0_0.1
- removed net DRIVER2:CW: DRIVER2:STHV_0.CW
- removed net DRIVER2:DVDD: DRIVER2:C182.1, DRIVER2:R2.2, DRIVER2:STHV_0.DVDD
- removed net DRIVER2:IN0_0: DRIVER2:STHV_0.IN1_0
- removed net DRIVER2:IN0_1: DRIVER2:STHV_0.IN1_1
- removed net DRIVER2:IN1_0: DRIVER2:STHV_0.IN2_0
- removed net DRIVER2:IN1_1: DRIVER2:STHV_0.IN2_1
- removed net DRIVER2:IN2_0: DRIVER2:STHV_0.IN3_0
- removed net DRIVER2:IN2_1: DRIVER2:STHV_0.IN3_1
- removed net DRIVER2:IN3_0: DRIVER2:STHV_0.IN4_0
- removed net DRIVER2:IN3_1: DRIVER2:STHV_0.IN4_1
- removed net DRIVER2:IN4_0: DRIVER2:STHV_0.IN5_0
- removed net DRIVER2:IN4_1: DRIVER2:STHV_0.IN5_1
- removed net DRIVER2:IN5_0: DRIVER2:STHV_0.IN6_0
- removed net DRIVER2:IN5_1: DRIVER2:STHV_0.IN6_1
- removed net DRIVER2:IN6_0: DRIVER2:STHV_0.IN7_0
- removed net DRIVER2:IN6_1: DRIVER2:STHV_0.IN7_1
- removed net DRIVER2:IN7_0: DRIVER2:STHV_0.IN8_0
- removed net DRIVER2:IN7_1: DRIVER2:STHV_0.IN8_1
- removed net DRIVER2:INX_1_0: DRIVER2:IN0_1.1
- removed net DRIVER2:LVOUT_0: DRIVER2:LVOUT0.1, DRIVER2:STHV_0.LVOUT_1
- removed net DRIVER2:LVOUT_1: DRIVER2:STHV_0.LVOUT_2
- removed net DRIVER2:LVOUT_2: DRIVER2:STHV_0.LVOUT_3
- removed net DRIVER2:LVOUT_3: DRIVER2:STHV_0.LVOUT_4
- removed net DRIVER2:LVOUT_4: DRIVER2:STHV_0.LVOUT_5
- removed net DRIVER2:LVOUT_5: DRIVER2:STHV_0.LVOUT_6
- removed net DRIVER2:LVOUT_6: DRIVER2:STHV_0.LVOUT_7
- removed net DRIVER2:LVOUT_7: DRIVER2:STHV_0.LVOUT_8
- removed net DRIVER2:OUT_0: DRIVER2:D0_0.A, DRIVER2:D0_1.C, DRIVER2:STHV_0.XDCR_1, DRIVER2:T_OUT_0.1
- removed net DRIVER2:OUT_1: DRIVER2:D1_0.A, DRIVER2:D1_1.C, DRIVER2:STHV_0.XDCR_2, DRIVER2:T_OUT_1.1
- removed net DRIVER2:OUT_2: DRIVER2:D2_0.A, DRIVER2:D2_1.C, DRIVER2:STHV_0.XDCR_3, DRIVER2:T_OUT_2.1
- removed net DRIVER2:OUT_3: DRIVER2:D3_0.A, DRIVER2:D3_1.C, DRIVER2:STHV_0.XDCR_4, DRIVER2:T_OUT_3.1
- removed net DRIVER2:OUT_4: DRIVER2:D4_0.A, DRIVER2:D4_1.C, DRIVER2:STHV_0.XDCR_5, DRIVER2:T_OUT_4.1
- removed net DRIVER2:OUT_5: DRIVER2:D5_0.A, DRIVER2:D5_1.C, DRIVER2:STHV_0.XDCR_6, DRIVER2:T_OUT_5.1
- removed net DRIVER2:OUT_6: DRIVER2:D6_0.A, DRIVER2:D6_1.C, DRIVER2:STHV_0.XDCR_7, DRIVER2:T_OUT_6.1
- removed net DRIVER2:OUT_7: DRIVER2:D7_0.A, DRIVER2:D7_1.C, DRIVER2:STHV_0.XDCR_8, DRIVER2:T_OUT_7.1
- removed net DRIVER2:PWM_INT0: DRIVER2:IN0_0.1
- removed net RECEIVER1:ADC2:ADIN2_N: RECEIVER1:ADC2:ADC1.5
- removed net RECEIVER1:ADC2:ADIN2_P: RECEIVER1:ADC2:ADC1.6
- removed net RECEIVER1:ADC2:ADIN3_N: RECEIVER1:ADC2:ADC1.3
- removed net RECEIVER1:ADC2:ADIN3_P: RECEIVER1:ADC2:ADC1.4
- removed net RECEIVER1:ADC2:ADIN4_N: RECEIVER1:ADC2:ADC1.1
- removed net RECEIVER1:ADC2:ADIN4_P: RECEIVER1:ADC2:ADC1.2
- removed net RECEIVER1:BUSY: RECEIVER1:ADC2:ADC1.26
- removed net RECEIVER1:CNV: RECEIVER1:ADC2:ADC1.15
- removed net RECEIVER1:S12:ENV1_N: RECEIVER1:S12:C78.1, RECEIVER1:S12:D6.A, RECEIVER1:S12:R44.2, RECEIVER1:S12:X12.2
- removed net RECEIVER1:S12:ENV1_P: RECEIVER1:S12:C77.1, RECEIVER1:S12:D5.C, RECEIVER1:S12:R43.2, RECEIVER1:S12:X12.1
- removed net RECEIVER1:S12:VO1_3: RECEIVER1:S12:SLIDESWITCH7.P$3, RECEIVER1:S12:SLIDESWITCH7.P$6
- removed net RECEIVER1:S12:VO1_3_N: RECEIVER1:S12:D6.C, RECEIVER1:S12:SLIDESWITCH7.P$5, RECEIVER1:S12:X2.2
- removed net RECEIVER1:S12:VO1_3_P: RECEIVER1:S12:D5.A, RECEIVER1:S12:SLIDESWITCH7.P$2, RECEIVER1:S12:X2.1
- removed net RECEIVER1:S1:5V: RECEIVER1:S1:L27.1, RECEIVER1:S1:L28.1, RECEIVER1:S1:L29.1, RECEIVER1:S1:L30.1, RECEIVER1:S1:L31.1, RECEIVER1:S1:L32.1, RECEIVER1:S1:R1.2, RECEIVER1:S1:R3.2, RECEIVER1:S1:SLIDESWITCH1.P$3, RECEIVER1:S1:SLIDESWITCH2.P$3
- removed net RECEIVER1:S1:LVOUT_0: RECEIVER1:S1:D1.3, RECEIVER1:S1:L1.1
- removed net RECEIVER1:S1:LVOUT_1: RECEIVER1:S1:D2.3, RECEIVER1:S1:L6.1
- removed net RECEIVER1:S1:N$10: RECEIVER1:S1:GAIN12_1.1
- removed net RECEIVER1:S1:N$7: RECEIVER1:S1:JP1.2, RECEIVER1:S1:R4.1
- removed net RECEIVER1:S1:N$8: RECEIVER1:S1:JP2.2, RECEIVER1:S1:R5.1
- removed net RECEIVER1:S1:N$9: RECEIVER1:S1:GAIN34_1.1
- removed net RECEIVER1:S1:R1_OUT_N: RECEIVER1:S1:C6.2
- removed net RECEIVER1:S1:R1_OUT_P: RECEIVER1:S1:C7.2
- removed net RECEIVER1:S1:R2_OUT_N: RECEIVER1:S1:C14.2
- removed net RECEIVER1:S1:R2_OUT_P: RECEIVER1:S1:C13.2
- removed net RECEIVER1:S1:VCM1: RECEIVER1:S1:IC1.50
- removed net RECEIVER1:S1:VCM2: RECEIVER1:S1:IC1.49
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