File: silense.sch (EAGLE design)
At the start: 0 parts

Commit message: schematic done except for power
Other:
- note added: "AD8334 - 2 Channels"
- note removed: "Channel 1,2"
- note removed: "TODO make ground symbols the same"
- note removed: "TODO: 5V Entry GND Entry 1V deduction with varistor with low pass network Other voltages?"
- note removed: "TODO: Power supplies"
- note removed: "todo: all vcm together?"
- note removed: "todo: attach to gnd or better solution? N$10 & N$9"
- note removed: "todo: can we reuse power supplies? todo: are names correct over multiple sheets?"
- note removed: "todo: change mode & hilo switches by resistor (easy to (de)solder)"
- note removed: "todo: change with appropriate envelope detection"
- note removed: "todo: check 5V: is it necessary or 3v3 also fine? => 3v3 comes from zedboard as well as powerconnboard"
- note removed: "todo: check footprint trimpots"
- note removed: "todo: check if we're converting against 2v5: stable voltage!"
